File: TheFalcon/PCB/TheFalcon[Left]/RGBArray.kicad_sch (KiCad schematic)
At the start: 59 parts, among them IC1 IS31FL3729-QFLS4-TR, J4 Conn_01x01

Commit message: Saving before I go crazy on PCB
Parts:
- removed J4: Conn_01x01, Connector_Wire:SolderWire-0.1sqmm_1x01_D0.4mm_OD1mm, symbol Connector_Generic:Conn_01x01
- removed R28: 0, Resistor_SMD:R_0805_2012Metric, symbol Device:R
- R10, R11, R12, R13, R14, R15, R16, R17, R18, R19, R20, R21, R22, R23, R5, R6, R9: footprint Resistor_SMD:R_0201_0603Metric -> Resistor_SMD:R_0603_1608Metric
Connections:
- net AD is gone; now on net GND: IC1.28 (AD)

Commit message: Save
Parts:
- RGB1, RGB10, RGB11, RGB12, RGB13, RGB14, RGB15, RGB16, RGB17, RGB18, RGB19, RGB2, RGB20, RGB21, RGB22, RGB23, RGB24, RGB25, RGB26, RGB27, RGB28, RGB29, RGB3, RGB30, RGB31, RGB32, RGB33, RGB34, RGB35, RGB37, RGB4, RGB5, RGB6, RGB7, RGB8, RGB9: footprint SamacSys_Parts:T36K3BGR05D000121U1930_MODEL -> SamacSys_Parts:T36K3BGR05D000121U1930_MODEL_INVERTED
Changed lines of the file:
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@@
 			)
 		)
-		(property "Footprint" "SamacSys_Parts:T36K3BGR05D000121U1930_MODEL"
+		(property "Footprint" "SamacSys_Parts:T36K3BGR05D000121U1930_MODEL_INVERTED"
 			(at -74.6 121.92 0)
 			(effects
@@
 			)
 		)
-		(property "Footprint" "SamacSys_Parts:T36K3BGR05D000121U1930_MODEL"
+		(property "Footprint" "SamacSys_Parts:T36K3BGR05D000121U1930_MODEL_INVERTED"
 			(at -54.28 55.88 0)
 			(effects
@@
 			)
 		)
-		(property "Footprint" "SamacSys_Parts:T36K3BGR05D000121U1930_MODEL"
+		(property "Footprint" "SamacSys_Parts:T36K3BGR05D000121U1930_MODEL_INVERTED"
 			(at -23.8 187.96 0)
 			(effects
@@
 			)
 		)
-		(property "Footprint" "SamacSys_Parts:T36K3BGR05D000121U1930_MODEL"
+		(property "Footprint" "SamacSys_Parts:T36K3BGR05D000121U1930_MODEL_INVERTED"
 			(at -3.48 187.96 0)
 			(effects
@@
 			)
 		)
-		(property "Footprint" "SamacSys_Parts:T36K3BGR05D000121U1930_MODEL"
+		(property "Footprint" "SamacSys_Parts:T36K3BGR05D000121U1930_MODEL_INVERTED"
 			(at -44.12 121.92 0)
 			(effects
@@
 			)
 		)
-		(property "Footprint" "SamacSys_Parts:T36K3BGR05D000121U1930_MODEL"
+		(property "Footprint" "SamacSys_Parts:T36K3BGR05D000121U1930_MODEL_INVERTED"
 			(at -44.12 187.96 0)
 			(effects
@@
 			)
 		)
-		(property "Footprint" "SamacSys_Parts:T36K3BGR05D000121U1930_MODEL"
+		(property "Footprint" "SamacSys_Parts:T36K3BGR05D000121U1930_MODEL_INVERTED"
 			(at -23.8 55.88 0)
 			(effects
@@
 			)
 		)
-		(property "Footprint" "SamacSys_Parts:T36K3BGR05D000121U1930_MODEL"
+		(property "Footprint" "SamacSys_Parts:T36K3BGR05D000121U1930_MODEL_INVERTED"
 			(at -74.6 154.94 0)
 			(effects
@@
 			)
 		)
-		(property "Footprint" "SamacSys_Parts:T36K3BGR05D000121U1930_MODEL"
+		(property "Footprint" "SamacSys_Parts:T36K3BGR05D000121U1930_MODEL_INVERTED"
 			(at -23.8 88.9 0)
 			(effects
@@
 			)
 		)
-		(property "Footprint" "SamacSys_Parts:T36K3BGR05D000121U1930_MODEL"
+		(property "Footprint" "SamacSys_Parts:T36K3BGR05D000121U1930_MODEL_INVERTED"
 			(at -64.44 187.96 0)
 			(effects
@@
 			)
 		)
-		(property "Footprint" "SamacSys_Parts:T36K3BGR05D000121U1930_MODEL"
+		(property "Footprint" "SamacSys_Parts:T36K3BGR05D000121U1930_MODEL_INVERTED"
 			(at -33.96 55.88 0)
 			(effects
@@
 			)
 		)
-		(property "Footprint" "SamacSys_Parts:T36K3BGR05D000121U1930_MODEL"
+		(property "Footprint" "SamacSys_Parts:T36K3BGR05D000121U1930_MODEL_INVERTED"
 			(at -23.8 121.92 0)
 			(effects
@@
 			)
 		)
-		(property "Footprint" "SamacSys_Parts:T36K3BGR05D000121U1930_MODEL"
+		(property "Footprint" "SamacSys_Parts:T36K3BGR05D000121U1930_MODEL_INVERTED"
 			(at -54.28 187.96 0)
 			(effects
@@
 			)
 		)
-		(property "Footprint" "SamacSys_Parts:T36K3BGR05D000121U1930_MODEL"
+		(property "Footprint" "SamacSys_Parts:T36K3BGR05D000121U1930_MODEL_INVERTED"
 			(at -13.64 55.88 0)
 			(effects
@@
 			)
 		)
-		(property "Footprint" "SamacSys_Parts:T36K3BGR05D000121U1930_MODEL"
+		(property "Footprint" "SamacSys_Parts:T36K3BGR05D000121U1930_MODEL_INVERTED"
 			(at -64.44 121.92 0)
 			(effects
@@
 			)
 		)
-		(property "Footprint" "SamacSys_Parts:T36K3BGR05D000121U1930_MODEL"
+		(property "Footprint" "SamacSys_Parts:T36K3BGR05D000121U1930_MODEL_INVERTED"
 			(at -44.12 88.9 0)
 			(effects
@@
 			)
 		)
-		(property "Footprint" "SamacSys_Parts:T36K3BGR05D000121U1930_MODEL"
+		(property "Footprint" "SamacSys_Parts:T36K3BGR05D000121U1930_MODEL_INVERTED"
 			(at -23.8 154.94 0)
 			(effects
@@
 			)
 		)
-		(property "Footprint" "SamacSys_Parts:T36K3BGR05D000121U1930_MODEL"
+		(property "Footprint" "SamacSys_Parts:T36K3BGR05D000121U1930_MODEL_INVERTED"
 			(at -74.6 88.9 0)
 			(effects
@@
 			)
 		)
-		(property "Footprint" "SamacSys_Parts:T36K3BGR05D000121U1930_MODEL"
+		(property "Footprint" "SamacSys_Parts:T36K3BGR05D000121U1930_MODEL_INVERTED"
 			(at -13.64 88.9 0)
 			(effects
@@
 			)
 		)
-		(property "Footprint" "SamacSys_Parts:T36K3BGR05D000121U1930_MODEL"
+		(property "Footprint" "SamacSys_Parts:T36K3BGR05D000121U1930_MODEL_INVERTED"
 			(at -44.12 55.88 0)
 			(effects
@@
 			)
 		)
-		(property "Footprint" "SamacSys_Parts:T36K3BGR05D000121U1930_MODEL"
+		(property "Footprint" "SamacSys_Parts:T36K3BGR05D000121U1930_MODEL_INVERTED"
 			(at -64.44 88.9 0)
 			(effects
@@
 			)
 		)
-		(property "Footprint" "SamacSys_Parts:T36K3BGR05D000121U1930_MODEL"
+		(property "Footprint" "SamacSys_Parts:T36K3BGR05D000121U1930_MODEL_INVERTED"
 			(at -74.6 187.96 0)
 			(effects
@@
 			)
 		)
-		(property "Footprint" "SamacSys_Parts:T36K3BGR05D000121U1930_MODEL"
+		(property "Footprint" "SamacSys_Parts:T36K3BGR05D000121U1930_MODEL_INVERTED"
 			(at -64.44 55.88 0)
 			(effects
@@
 			)
 		)
-		(property "Footprint" "SamacSys_Parts:T36K3BGR05D000121U1930_MODEL"
+		(property "Footprint" "SamacSys_Parts:T36K3BGR05D000121U1930_MODEL_INVERTED"
 			(at -64.44 154.94 0)
 			(effects
@@
 			)
 		)
-		(property "Footprint" "SamacSys_Parts:T36K3BGR05D000121U1930_MODEL"
+		(property "Footprint" "SamacSys_Parts:T36K3BGR05D000121U1930_MODEL_INVERTED"
 			(at -44.12 154.94 0)
 			(effects
@@
 			)
 		)
-		(property "Footprint" "SamacSys_Parts:T36K3BGR05D000121U1930_MODEL"
+		(property "Footprint" "SamacSys_Parts:T36K3BGR05D000121U1930_MODEL_INVERTED"
 			(at -13.64 154.94 0)
 			(effects
@@
 			)
 		)
-		(property "Footprint" "SamacSys_Parts:T36K3BGR05D000121U1930_MODEL"
+		(property "Footprint" "SamacSys_Parts:T36K3BGR05D000121U1930_MODEL_INVERTED"
 			(at -33.96 88.9 0)
 			(effects
@@
 			)
 		)
-		(property "Footprint" "SamacSys_Parts:T36K3BGR05D000121U1930_MODEL"
+		(property "Footprint" "SamacSys_Parts:T36K3BGR05D000121U1930_MODEL_INVERTED"
 			(at -33.96 187.96 0)
 			(effects
@@
 			)
 		)
-		(property "Footprint" "SamacSys_Parts:T36K3BGR05D000121U1930_MODEL"
+		(property "Footprint" "SamacSys_Parts:T36K3BGR05D000121U1930_MODEL_INVERTED"
 			(at -33.96 154.94 0)
 			(effects
@@
 			)
 		)
-		(property "Footprint" "SamacSys_Parts:T36K3BGR05D000121U1930_MODEL"
+		(property "Footprint" "SamacSys_Parts:T36K3BGR05D000121U1930_MODEL_INVERTED"
 			(at -33.96 121.92 0)
 			(effects
@@
 			)
 		)
-		(property "Footprint" "SamacSys_Parts:T36K3BGR05D000121U1930_MODEL"
+		(property "Footprint" "SamacSys_Parts:T36K3BGR05D000121U1930_MODEL_INVERTED"
 			(at -13.64 121.92 0)
 			(effects
@@
 			)
 		)
-		(property "Footprint" "SamacSys_Parts:T36K3BGR05D000121U1930_MODEL"
+		(property "Footprint" "SamacSys_Parts:T36K3BGR05D000121U1930_MODEL_INVERTED"
 			(at -13.64 187.96 0)
 			(effects
@@
 			)
 		)
-		(property "Footprint" "SamacSys_Parts:T36K3BGR05D000121U1930_MODEL"
+		(property "Footprint" "SamacSys_Parts:T36K3BGR05D000121U1930_MODEL_INVERTED"
 			(at -54.28 88.9 0)
 			(effects
@@
 			)
 		)
-		(property "Footprint" "SamacSys_Parts:T36K3BGR05D000121U1930_MODEL"
+		(property "Footprint" "SamacSys_Parts:T36K3BGR05D000121U1930_MODEL_INVERTED"
 			(at -54.28 121.92 0)
 			(effects
@@
 			)
 		)
-		(property "Footprint" "SamacSys_Parts:T36K3BGR05D000121U1930_MODEL"
+		(property "Footprint" "SamacSys_Parts:T36K3BGR05D000121U1930_MODEL_INVERTED"
 			(at -74.6 55.88 0)
 			(effects
@@
 			)
 		)
-		(property "Footprint" "SamacSys_Parts:T36K3BGR05D000121U1930_MODEL"
+		(property "Footprint" "SamacSys_Parts:T36K3BGR05D000121U1930_MODEL_INVERTED"
 			(at -54.28 154.94 0)
 			(effects

Commit message: Save
Connections:
- net SW1: now also RGB37.2 (COM_A); no longer RGB1.2 (COM_A), RGB15.2 (COM_A), RGB22.2 (COM_A), RGB29.2 (COM_A), RGB8.2 (COM_A)
- net SW2: now also RGB14.2 (COM_A), RGB21.2 (COM_A), RGB28.2 (COM_A), RGB35.2 (COM_A), RGB7.2 (COM_A); no longer RGB16.2 (COM_A), RGB2.2 (COM_A), RGB23.2 (COM_A), RGB30.2 (COM_A), RGB9.2 (COM_A)
- net SW3: now also RGB13.2 (COM_A), RGB20.2 (COM_A), RGB27.2 (COM_A), RGB34.2 (COM_A), RGB6.2 (COM_A); no longer RGB10.2 (COM_A), RGB17.2 (COM_A), RGB24.2 (COM_A), RGB3.2 (COM_A), RGB31.2 (COM_A)
- net SW4: now also RGB12.2 (COM_A), RGB19.2 (COM_A), RGB26.2 (COM_A), RGB33.2 (COM_A), RGB5.2 (COM_A); no longer RGB11.2 (COM_A), RGB18.2 (COM_A), RGB25.2 (COM_A), RGB32.2 (COM_A), RGB4.2 (COM_A)
- net SW5: now also RGB11.2 (COM_A), RGB18.2 (COM_A), RGB25.2 (COM_A), RGB32.2 (COM_A), RGB4.2 (COM_A); no longer RGB12.2 (COM_A), RGB19.2 (COM_A), RGB26.2 (COM_A), RGB33.2 (COM_A), RGB5.2 (COM_A)
- net SW6: now also RGB10.2 (COM_A), RGB17.2 (COM_A), RGB24.2 (COM_A), RGB3.2 (COM_A), RGB31.2 (COM_A); no longer RGB13.2 (COM_A), RGB20.2 (COM_A), RGB27.2 (COM_A), RGB34.2 (COM_A), RGB6.2 (COM_A)
- net SW7: now also RGB16.2 (COM_A), RGB2.2 (COM_A), RGB23.2 (COM_A), RGB30.2 (COM_A), RGB9.2 (COM_A); no longer RGB14.2 (COM_A), RGB21.2 (COM_A), RGB28.2 (COM_A), RGB35.2 (COM_A), RGB7.2 (COM_A)
- net SW8: now also RGB1.2 (COM_A), RGB15.2 (COM_A), RGB22.2 (COM_A), RGB29.2 (COM_A), RGB8.2 (COM_A); no longer RGB37.2 (COM_A)
Changed lines of the file:
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@@
+		)
+	)
+	(label "SW2"
+		(at 74.93 27.94 0)
+		(effects
+			(font
+				(size 1.27 1.27)
+			)
+			(justify left bottom)
+		)
+	)
+	(label "SW4"
+		(at 54.61 27.94 0)
+		(effects
+			(font
+				(size 1.27 1.27)
+			)
+			(justify left bottom)
 		)
 	)
@@
 		)
 	)
+	(label "SW8"
+		(at 13.97 27.94 0)
+		(effects
+			(font
+				(size 1.27 1.27)
+			)
+			(justify left bottom)
+		)
+	)
 	(label "CS7"
 		(at 170.18 66.04 180)
@@
 		)
 	)
-	(label "SW3"
-		(at 34.29 27.94 0)
-		(effects
-			(font
-				(size 1.27 1.27)
-			)
-			(justify left bottom)
-		)
-	)
 	(label "CS15"
 		(at 110.49 194.31 0)
@@
 		)
 	)
+	(label "SW7"
+		(at 24.13 27.94 0)
+		(effects
+			(font
+				(size 1.27 1.27)
+			)
+			(justify left bottom)
+		)
+	)
 	(label "CS12"
 		(at 111.76 161.29 0)
@@
 		)
 	)
-	(label "SW6"
+	(label "SW3"
 		(at 64.77 27.94 0)
 		(effects
@@
 		)
 	)
-	(label "SW4"
-		(at 44.45 27.94 0)
-		(effects
-			(font
-				(size 1.27 1.27)
-			)
-			(justify left bottom)
-		)
-	)
 	(label "CS3"
 		(at 104.14 62.23 0)
@@
 		)
 	)
+	(label "SW1"
+		(at 85.09 27.94 0)
+		(effects
+			(font
+				(size 1.27 1.27)
+			)
+			(justify left bottom)
+		)
+	)
 	(label "CS4"
 		(at 104.14 67.31 0)
@@
 		)
 	)
-	(label "SW5"
-		(at 54.61 27.94 0)
-		(effects
-			(font
-				(size 1.27 1.27)
-			)
-			(justify left bottom)
-		)
-	)
 	(label "CS5"
 		(at 170.18 60.96 180)
@@
 		)
 	)
+	(label "SW6"
+		(at 34.29 27.94 0)
+		(effects
+			(font
+				(size 1.27 1.27)
+			)
+			(justify left bottom)
+		)
+	)
 	(label "B_RGB_ROW_4"
 		(at 96.52 165.1 0)
@@
 		)
 	)
-	(label "SW2"
-		(at 24.13 27.94 0)
-		(effects
-			(font
-				(size 1.27 1.27)
-			)
-			(justify left bottom)
-		)
-	)
 	(label "CS2"
 		(at 184.15 38.1 270)
@@
 		)
 	)
-	(label "SW8"
-		(at 85.09 27.94 0)
-		(effects
-			(font
-				(size 1.27 1.27)
-			)
-			(justify left bottom)
-		)
-	)
 	(label "B_RGB_ROW_0"
 		(at 90.17 30.48 0)
@@
 		)
 	)
+	(label "SW5"
+		(at 44.45 27.94 0)
+		(effects
+			(font
+				(size 1.27 1.27)
+			)
+			(justify left bottom)
+		)
+	)
 	(label "CS8"
 		(at 110.49 125.73 0)
@@
 		)
 	)
-	(label "SW7"
-		(at 74.93 27.94 0)
-		(effects
-			(font
-				(size 1.27 1.27)
-			)
-			(justify left bottom)
-		)
-	)
 	(label "CS15"
 		(at 189.23 100.33 90)
@@
 		(effects
 			(font
-				(size 1.27 1.27)
-			)
-			(justify left bottom)
-		)
-	)
-	(label "SW1"
-		(at 13.97 27.94 0)
-		(effects
-			(font

Commit message: Cleaning up
I have all connections, just cleaning up
Connections:
- net CS13: now also R17.2; no longer R23.2
- net CS14: now also R15.2; no longer R21.2
- net CS15: now also R16.2; no longer R22.2
- net CS7: now also R23.2; no longer R17.2
- net CS8: now also R21.2; no longer R15.2
- net CS9: now also R22.2; no longer R16.2
Changed lines of the file:
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@@
 	(wire
 		(pts
-			(xy 107.95 125.73) (xy 110.49 125.73)
+			(xy 107.95 125.73) (xy 111.76 125.73)
 		)
 		(stroke
@@
 	)
 	(label "CS13"
-		(at 111.76 167.64 0)
+		(at 115.57 96.52 0)
 		(effects
 			(font
@@
 	)
 	(label "CS15"
-		(at 110.49 194.31 0)
+		(at 111.76 128.27 0)
 		(effects
 			(font
@@
 	)
 	(label "CS7"
-		(at 115.57 96.52 0)
+		(at 111.76 167.64 0)
 		(effects
 			(font
@@
 	)
 	(label "CS8"
-		(at 110.49 125.73 0)
+		(at 110.49 191.77 0)
 		(effects
 			(font
@@
 	)
 	(label "CS14"
-		(at 110.49 191.77 0)
+		(at 111.76 125.73 0)
 		(effects
 			(font
@@
 	)
 	(label "CS9"
-		(at 111.76 128.27 0)
+		(at 110.49 194.31 0)
 		(effects
 			(font

Commit message: Save
Other:
- note removed: "Header pin to solder AD to change address"
Changed lines of the file:
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@@
-		)
-	)
-	(text "Header pin to solder AD \nto change address"
-		(exclude_from_sim no)
-		(at 242.57 50.292 0)
-		(effects
-			(font
-				(size 1.27 1.27)
-			)
 		)
 	)

Commit message: Files ready for production
Going to panelise seperate files to reduce PCBA cost
Parts:
- C12, C14: LCSC Part Number (none) -> C1525
- C13: LCSC Part Number (none) -> C1592
- IC1: Arrow Part Number IS31FL3729-QFLS4-TR -> (none); Arrow Price/Stock https://www.arrow.com/en/products/is31fl3729-qfls4-tr/integ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 -> (none); Height 0.8 -> (none); LCSC Part Number (none) -> C2940549; Manufacturer_Name Lumissil Microsystems -> (none); Manufacturer_Part_Number IS31FL3729-QFLS4-TR -> (none); Mouser Part Number 870-IS31FL3729QFLS4T -> (none); Mouser Price/Stock https://www.mouser.com/Search/Refine.aspx?Keyword=870-IS31F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 -> (none)
- R10, R12, R14, R15, R17, R18, R20, R21, R23, R9: LCSC Part Number (none) -> C22950
- R11, R13, R16, R19, R22: LCSC Part Number (none) -> C17738
- R5: LCSC Part Number (none) -> C14675
- R6: LCSC Part Number (none) -> C15401
- RGB1, RGB10, RGB11, RGB12, RGB13, RGB14, RGB15, RGB16, RGB17, RGB18, RGB19, RGB2, RGB20, RGB21, RGB22, RGB23, RGB24, RGB25, RGB26, RGB27, RGB28, RGB29, RGB3, RGB30, RGB31, RGB32, RGB33, RGB34, RGB35, RGB37, RGB4, RGB5, RGB6, RGB7, RGB8, RGB9: Height 1.95 -> (none); Link https://www.digikey.co.za/en/products/detail/harvatek-corpo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 -> (none); Manufacturer_Name Harvatek -> (none); Manufacturer_Part_Number T36K3BGR-05D000121U1930 -> (none)
