File: TheFalcon/PCB/TheFalcon[Left]/TheFalcon[Left].kicad_pcb (KiCad board)
At the start: 2 copper layers, 186 parts, among them IC1 IS31FL3729-QFLS4-TR, J1 Conn_01x04_Pin, J2 Conn_02x05_Odd_Even, J3 Conn_01x04_Pin, J4 Conn_01x01, J5 Conn_01x01, J6 Conn_01x01, SW1 SW_Push, SW2 SW_Push, SW3 SW_DIP_x02, U2 USBLC6-2P6, U3 USBLC6-2P6, U4 AMS1117-3.3, U5 USBLC6-2P6, U6 STM32G431CBTx, Y1 X322516MOB4SI

Commit message: Save
Parts:
- removed D34, D35: Diode, Diode_SMD:D_SOD-123
- removed D39: LED, LED_SMD:LED_0805_2012Metric
- removed J1: Conn_01x04_Pin, Connector_PinSocket_2.54mm:PinSocket_1x04_P2.54mm_Vertical
- removed J4, J5, J6: Conn_01x01, Connector_Wire:SolderWire-0.1sqmm_1x01_D0.4mm_OD1mm
- removed RGB36, RGB38: T36K3BGR-05D000121U1930, SamacSys_Parts:T36K3BGR05D000121U1930
- removed S37, S38: Keyswitch, Gateron_KS33_Hotswap:Gateron-KS33-Hotswap-1.5U
- removed USB1, USB2: USB_C_Receptacle_USB2.0_16P, Connector_USB:USB_C_Receptacle_G-Switch_GT-USB-7010ASV
- added 3V3: Conn_01x01, Connector_Wire:SolderWire-0.1sqmm_1x01_D0.4mm_OD1mm, B.Cu at (59.1, 30.3)
- added 5V/AD  Conn: Conn_01x01, Connector_Wire:SolderWire-0.1sqmm_1x01_D0.4mm_OD1mm, B.Cu at (115.3, 29.0)
- added GND: Conn_01x01, Connector_Wire:SolderWire-0.1sqmm_1x01_D0.4mm_OD1mm, B.Cu at (66.5, 30.1)
- added PWR: LED, LED_SMD:LED_0805_2012Metric, B.Cu at (63.2, 30.8)
- added Serial/I2C : USB_C_Receptacle_USB2.0_16P, Connector_USB:USB_C_Receptacle_G-Switch_GT-USB-7010ASV, B.Cu at (166.2, 29.2)
- added USB Connection: USB_C_Receptacle_USB2.0_16P, Connector_USB:USB_C_Receptacle_G-Switch_GT-USB-7010ASV, B.Cu at (37.8, 28.4)
- C1, C10, C11, C13, C15, C16, C17, C7, D1, D10, D11, D12, D13, D14, D15, D16, D17, D18, D19, D2, D20, D21, D22, D23, D24, D25, D26, D27, D28, D29, D3, D30, D31, D32, D33, D36, D37, D38, D4, D5, D6, D7, D8, D9, F1, IC1, R1, R10, R11, R12, R13, R14, R15, R16, R17, R18, R19, R2, R20, R21, R22, R23, R24, R25, R28, R29, R3, R30, R31, R32, R33, R4, R5, R6, R9, SW1, SW2, SW3, U2, U3, U4, U5, U6, Y1: moved to B.Cu
- C12, C14, C2, C3, C4, C5, C6, C8, C9: footprint Capacitor_SMD:C_0603_1608Metric -> Capacitor_SMD:C_0402_1005Metric; moved to B.Cu
- H1, H2, H3, H5, H6: footprint MountingHole:MountingHole_3.2mm_M3_Pad_Via -> MountingHole:MountingHole_2.2mm_M2_Pad; moved to B.Cu
- H4: footprint MountingHole:MountingHole_3.2mm_M3_Pad_Via -> MountingHole:MountingHole_2.2mm_M2_Pad
- J2: value Conn_02x05_Odd_Even -> Conn_01x04_Pin; footprint Connector_PinSocket_2.54mm:PinSocket_2x05_P2.54mm_Vertical -> Connector_Wire:SolderWire-1sqmm_1x04_P5.4mm_D1.4mm_OD2.7mm
- J3: footprint Connector_PinSocket_2.54mm:PinSocket_1x04_P2.54mm_Vertical -> Connector_Wire:SolderWire-1sqmm_1x04_P5.4mm_D1.4mm_OD2.7mm; moved to B.Cu
- RGB1, RGB10, RGB11, RGB12, RGB13, RGB14, RGB15, RGB16, RGB17, RGB18, RGB19, RGB2, RGB20, RGB21, RGB22, RGB23, RGB24, RGB25, RGB26, RGB27, RGB28, RGB29, RGB3, RGB30, RGB31, RGB32, RGB33, RGB34, RGB35, RGB37, RGB4, RGB5, RGB6, RGB7, RGB8, RGB9: footprint SamacSys_Parts:T36K3BGR05D000121U1930 -> SamacSys_Parts:T36K3BGR05D000121U1930_MODEL
- S1, S10, S11, S12, S13, S14, S15, S16, S17, S18, S19, S2, S20, S21, S22, S23, S24, S25, S26, S27, S28, S29, S3, S30, S31, S32, S33, S34, S4, S5, S6, S7, S8, S9: footprint Gateron_KS33_Hotswap:Gateron-KS33-Hotswap-1U -> Gateron_KS33_Hotswap:Gateron-KS33-Hotswap-1U_Model; moved to B.Cu
- S35, S36: footprint Gateron_KS33_Hotswap:Gateron-KS33-Hotswap-1U -> Gateron_KS33_Hotswap:Gateron-KS33-Hotswap-1.5U; moved to B.Cu
- moved D22 391.8 mm to (23.8, 104.8), turned to 90 degrees
- moved D29 391.0 mm to (23.8, 123.8), turned to 90 degrees
- moved D15 381.6 mm to (23.8, 85.7), turned to 90 degrees
- moved D8 373.5 mm to (23.8, 66.7), turned to 90 degrees
- moved D1 373.5 mm to (23.8, 47.6), turned to 90 degrees
- moved U2 373.1 mm to (37.9, 35.1), turned to -90 degrees
- moved D23 372.5 mm to (42.9, 104.8), turned to 90 degrees
- moved C10 372.1 mm to (47.0, 34.8), turned to -90 degrees
- moved D30 371.7 mm to (42.9, 123.8), turned to 90 degrees
- moved F1 369.9 mm to (45.5, 31.3)
- moved R2 368.9 mm to (29.9, 31.8), turned to -90 degrees
- moved H6 367.9 mm to (26.0, 37.0), turned to 180 degrees
- moved R1 366.6 mm to (31.5, 31.8), turned to -90 degrees
- moved D16 362.3 mm to (42.9, 85.7), turned to 90 degrees
- moved C11 361.0 mm to (60.2, 34.2), turned to -90 degrees
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Connections:
- J2 pad 1: +3.3V -> SYS_JTAG_SWDIO
- J2 pad 2: SYS_JTAG_SWDIO -> SYS_JTAG_SWCLK
- J2 pad 3: GND -> SYS_JTAG_TRACE
- J2 pad 4: SYS_JTAG_SWCLK -> NRST
- R13 pad 1: /RGB Array/R_RGB_ROW_0 -> /RGB Array/R_RGB_ROW_1
- R16 pad 1: /RGB Array/R_RGB_ROW_0 -> /RGB Array/R_RGB_ROW_2
- R19 pad 1: /RGB Array/R_RGB_ROW_0 -> /RGB Array/R_RGB_ROW_3
- R22 pad 1: /RGB Array/R_RGB_ROW_0 -> /RGB Array/R_RGB_ROW_4
- RGB10 pad 1: /RGB Array/R_RGB_ROW_0 -> /RGB Array/R_RGB_ROW_1
- RGB11 pad 1: /RGB Array/R_RGB_ROW_0 -> /RGB Array/R_RGB_ROW_1
- RGB12 pad 1: /RGB Array/R_RGB_ROW_0 -> /RGB Array/R_RGB_ROW_1
- RGB13 pad 1: /RGB Array/R_RGB_ROW_0 -> /RGB Array/R_RGB_ROW_1
- RGB14 pad 1: /RGB Array/R_RGB_ROW_0 -> /RGB Array/R_RGB_ROW_1
- RGB15 pad 1: /RGB Array/R_RGB_ROW_0 -> /RGB Array/R_RGB_ROW_2
- RGB16 pad 1: /RGB Array/R_RGB_ROW_0 -> /RGB Array/R_RGB_ROW_2
- RGB17 pad 1: /RGB Array/R_RGB_ROW_0 -> /RGB Array/R_RGB_ROW_2
- RGB18 pad 1: /RGB Array/R_RGB_ROW_0 -> /RGB Array/R_RGB_ROW_2
- RGB19 pad 1: /RGB Array/R_RGB_ROW_0 -> /RGB Array/R_RGB_ROW_2
- RGB20 pad 1: /RGB Array/R_RGB_ROW_0 -> /RGB Array/R_RGB_ROW_2
- RGB21 pad 1: /RGB Array/R_RGB_ROW_0 -> /RGB Array/R_RGB_ROW_2
- RGB22 pad 1: /RGB Array/R_RGB_ROW_0 -> /RGB Array/R_RGB_ROW_3
- RGB23 pad 1: /RGB Array/R_RGB_ROW_0 -> /RGB Array/R_RGB_ROW_3
- RGB24 pad 1: /RGB Array/R_RGB_ROW_0 -> /RGB Array/R_RGB_ROW_3
- RGB25 pad 1: /RGB Array/R_RGB_ROW_0 -> /RGB Array/R_RGB_ROW_3
- RGB26 pad 1: /RGB Array/R_RGB_ROW_0 -> /RGB Array/R_RGB_ROW_3
- RGB27 pad 1: /RGB Array/R_RGB_ROW_0 -> /RGB Array/R_RGB_ROW_3
- RGB28 pad 1: /RGB Array/R_RGB_ROW_0 -> /RGB Array/R_RGB_ROW_3
- RGB29 pad 1: /RGB Array/R_RGB_ROW_0 -> /RGB Array/R_RGB_ROW_4
- RGB30 pad 1: /RGB Array/R_RGB_ROW_0 -> /RGB Array/R_RGB_ROW_4
- RGB31 pad 1: /RGB Array/R_RGB_ROW_0 -> /RGB Array/R_RGB_ROW_4
- RGB32 pad 1: /RGB Array/R_RGB_ROW_0 -> /RGB Array/R_RGB_ROW_4
- RGB33 pad 1: /RGB Array/R_RGB_ROW_0 -> /RGB Array/R_RGB_ROW_4
- RGB34 pad 1: /RGB Array/R_RGB_ROW_0 -> /RGB Array/R_RGB_ROW_4
- RGB35 pad 1: /RGB Array/R_RGB_ROW_0 -> /RGB Array/R_RGB_ROW_4
- RGB37 pad 1: /RGB Array/R_RGB_ROW_0 -> /RGB Array/R_RGB_ROW_4
- RGB8 pad 1: /RGB Array/R_RGB_ROW_0 -> /RGB Array/R_RGB_ROW_1
- RGB9 pad 1: /RGB Array/R_RGB_ROW_0 -> /RGB Array/R_RGB_ROW_1
- S34 pad 1: Col5 -> Col4
- S34 pad 2: Net-(D34-A) -> Net-(D36-A)
- S35 pad 1: Col6 -> Col5
- S35 pad 2: Net-(D35-A) -> Net-(D37-A)
- S36 pad 1: Col4 -> Col6
- S36 pad 2: Net-(D36-A) -> Net-(D38-A)
- U6 pad 22: BOOT_Tx+ -> unconnected-(U6-PB10-Pad22)
- U6 pad 25: BOOT_Tx- -> unconnected-(U6-PB11-Pad25)
Other:
- board outline added: 171.1 x 139.5 mm
- board text added: "For Instructional Use Only."
- board text added: "SOLIDWORKS Educational Product."

Commit message: Save
Parts:
- J4: renamed from 5V/AD  Conn
- USB1: renamed from USB Connection
- USB2: renamed from Serial/I2C 
- moved C6 120.9 mm to (36.5, 70.2), turned to 180 degrees
- moved C5 120.8 mm to (47.1, 77.3)
- moved C8 120.6 mm to (37.8, 71.7)
- moved C2 120.5 mm to (37.9, 68.7)
- moved C16 120.4 mm to (43.1, 83.4)
- moved R33 120.3 mm to (44.1, 63.8), turned to 0 degrees
- moved R24 120.3 mm to (43.4, 64.6), turned to 180 degrees
- moved U6 120.2 mm to (43.9, 71.5)
- moved C7 120.2 mm to (34.4, 71.3)
- moved C15 120.2 mm to (45.2, 83.4)
- moved C3 120.0 mm to (49.7, 74.0)
- moved C1 120.0 mm to (51.4, 74.2)
- moved C4 119.9 mm to (46.7, 65.6)
- moved C17 119.7 mm to (36.4, 72.2)
- moved Y1 119.6 mm to (45.2, 86.7)
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- renumbered PWR to D39, 3V3 to J5, GND to J6
Connections:
- J3 pad 1: PB12 -> PB10
- J3 pad 4: PB15 -> PC13
- U2 pad 1: USB_CONN_D+ -> USB_MCU_D+
- U2 pad 3: USB_CONN_D- -> USB_MCU_D-
- U2 pad 4: USB_MCU_D- -> USB_CONN_D-
- U2 pad 6: USB_MCU_D+ -> USB_CONN_D+
- U3 pad 1: USB_CONN_Tx+ -> USB_Tx-
- U3 pad 3: UBS_CONN_Tx- -> USB_Tx+
- U3 pad 4: USB_Tx+ -> USB_CONN_Tx-
- U3 pad 6: USB_Tx- -> USB_CONN_Tx+
- U6 pad 13: Row0 -> Row2
- U6 pad 14: Row1 -> Row3
- U6 pad 15: Row2 -> Row4
- U6 pad 16: Row3 -> PB10
- U6 pad 17: Row4 -> unconnected-(U6-PB1-Pad17)
- U6 pad 2: Col0 -> PC13
- U6 pad 25: unconnected-(U6-PB11-Pad25) -> Row1
- U6 pad 26: PB12 -> Row0
- U6 pad 29: PB15 -> Col0
- U6 pad 4: Col2 -> unconnected-(U6-PC15-Pad4)
- U6 pad 8: unconnected-(U6-PA0-Pad8) -> Col2
- USB2 pad A7: UBS_CONN_Tx- -> USB_CONN_Tx-
- USB2 pad B7: UBS_CONN_Tx- -> USB_CONN_Tx-
Routing:
- net Col6: track 0.00 -> 319.4 mm
- net Col5: track 0.00 -> 292.8 mm
- net Col4: track 0.00 -> 281.8 mm, vias 0 -> 2
- net Col3: track 0.00 -> 232.6 mm, vias 0 -> 4
- net Col2: track 0.00 -> 208.3 mm, vias 0 -> 2
- net Row1: track 0.00 -> 204.3 mm, vias 0 -> 18
- net Row3: track 0.00 -> 191.5 mm, vias 0 -> 14
- net Row2: track 0.00 -> 169.3 mm, vias 0 -> 16
- net Row0: track 0.00 -> 165.8 mm, vias 0 -> 12
- net Row4: track 0.00 -> 164.3 mm, vias 0 -> 2
- net ThumbRow: track 0.00 -> 153.9 mm, vias 0 -> 10
- net Col0: track 0.00 -> 140.4 mm, vias 0 -> 2
- net +3.3V: track 0.00 -> 139.0 mm, vias 0 -> 15
- net +5V: track 0.00 -> 138.5 mm, vias 0 -> 4
- net VBUS: track 0.00 -> 119.1 mm, vias 0 -> 2
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- added copper zone on B.Cu, net +3.3V
- added copper zone on B.Cu, net +5V
- added copper zone on B.Cu, net GND
- added copper zone on F.Cu, net GND
- added copper zone on B.Cu, net VBUS
Other:
- board size 171.1 x 139.5 mm -> 172.3 x 139.5 mm
- board text removed: "For Instructional Use Only."
- board text removed: "SOLIDWORKS Educational Product."

Commit message: Save
Parts:
- removed J4: Conn_01x01, Connector_Wire:SolderWire-0.1sqmm_1x01_D0.4mm_OD1mm
- removed R28, R29, R30, R31, R32: 0, Resistor_SMD:R_0805_2012Metric
- removed SW3: SW_DIP_x02, Button_Switch_SMD:SW_DIP_SPSTx02_Slide_KingTek_DSHP02TS_W7.62mm_P1.27mm
- removed U5: USBLC6-2P6, Package_TO_SOT_SMD:SOT-666
- H4, J2: moved to B.Cu
- R10, R11, R12, R13, R14, R15, R16, R17, R18, R19, R20, R21, R22, R23, R24, R25, R33, R5, R6, R9: footprint Resistor_SMD:R_0201_0603Metric -> Resistor_SMD:R_0603_1608Metric
- RGB1, RGB10, RGB11, RGB12, RGB13, RGB14, RGB15, RGB16, RGB17, RGB18, RGB19, RGB2, RGB20, RGB21, RGB22, RGB23, RGB24, RGB25, RGB26, RGB27, RGB28, RGB29, RGB3, RGB30, RGB31, RGB32, RGB33, RGB34, RGB35, RGB37, RGB4, RGB5, RGB6, RGB7, RGB9: footprint SamacSys_Parts:T36K3BGR05D000121U1930_MODEL -> SamacSys_Parts:T36K3BGR05D000121U1930_MODEL_INVERTED
- RGB8: footprint SamacSys_Parts:T36K3BGR05D000121U1930_MODEL -> SamacSys_Parts:T36K3BGR05D000121U1930_MODEL_INVERTED; moved to B.Cu
- moved RGB22 224.4 mm to (248.3, 44.2)
- moved RGB29 218.8 mm to (248.3, 85.5)
- moved RGB15 205.9 mm to (237.7, 61.9)
- moved RGB31 205.9 mm to (258.9, 38.3)
- moved RGB23 204.4 mm to (248.3, 50.1)
- moved RGB30 199.0 mm to (248.3, 91.4)
- moved RGB16 186.2 mm to (237.7, 67.8)
- moved D1 185.8 mm to (205.0, 100.9), turned to 180 degrees
- moved RGB32 184.1 mm to (258.9, 44.2)
- moved RGB24 183.1 mm to (248.3, 56.0)
- moved J2 180.2 mm to (201.1, 37.8), turned to 180 degrees
- moved D8 180.1 mm to (204.9, 97.6), turned to 180 degrees
- moved H3 178.9 mm to (183.1, 47.9)
- moved C7 174.8 mm to (205.8, 36.6), turned to 180 degrees
- moved RGB9 174.6 mm to (227.1, 85.5)
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Connections:
- IC1 pad 28: /RGB Array/AD -> GND
- USB2 pad A5: Net-(USB2-CC1) -> unconnected-(USB2-CC1-PadA5)
- USB2 pad A8: Net-(USB2-SBU1) -> unconnected-(USB2-SBU1-PadA8)
- USB2 pad B5: Net-(USB2-CC2) -> unconnected-(USB2-CC2-PadB5)
- USB2 pad B8: Net-(USB2-SBU2) -> unconnected-(USB2-SBU2-PadB8)
Routing:
- net Col6: track 319.4 -> 0.00 mm
- net Col5: track 292.8 -> 0.00 mm
- net Col4: track 281.8 -> 0.00 mm, vias 2 -> 0
- net Col3: track 232.6 -> 0.00 mm, vias 4 -> 0
- net Col2: track 208.3 -> 0.00 mm, vias 2 -> 0
- net Row1: track 204.3 -> 0.00 mm, vias 18 -> 0
- net Row3: track 191.5 -> 0.00 mm, vias 14 -> 0
- net Row2: track 169.3 -> 0.00 mm, vias 16 -> 0
- net Row0: track 165.8 -> 0.00 mm, vias 12 -> 0
- net Row4: track 164.3 -> 0.00 mm, vias 2 -> 0
- net ThumbRow: track 153.9 -> 0.00 mm, vias 10 -> 0
- net Col0: track 140.4 -> 0.00 mm, vias 2 -> 0
- net +3.3V: track 139.0 -> 0.00 mm, vias 15 -> 0
- net +5V: track 138.5 -> 0.00 mm, vias 4 -> 0
- net VBUS: track 119.1 -> 0.00 mm, vias 2 -> 0
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- removed copper zone on B.Cu, net +3.3V
- removed copper zone on B.Cu, net +5V
- removed copper zone on B.Cu, net GND
- removed copper zone on F.Cu, net GND
- removed copper zone on B.Cu, net VBUS
Other:
- board size 172.3 x 139.5 mm -> 173.3 x 142.5 mm

Commit message: Save
Parts:
- RGB8: moved to F.Cu
- moved RGB22 223.9 mm to (34.2, 109.8)
- moved RGB29 218.7 mm to (34.0, 129.0)
- moved RGB31 205.7 mm to (72.0, 124.2)
- moved RGB15 205.5 mm to (34.2, 91.0)
- moved RGB23 204.3 mm to (53.0, 110.0)
- moved R23 203.7 mm to (28.3, 132.7), turned to -90 degrees
- moved RGB30 198.9 mm to (53.0, 129.0)
- moved R20 198.6 mm to (28.4, 112.9), turned to -90 degrees
- moved R21 195.8 mm to (39.5, 132.2), turned to -90 degrees
- moved R22 193.3 mm to (41.0, 132.2), turned to -90 degrees
- moved R17 193.2 mm to (28.4, 93.8), turned to -90 degrees
- moved R9 193.1 mm to (26.9, 52.9), turned to -90 degrees
- moved R14 192.1 mm to (26.8, 73.4), turned to -90 degrees
- moved D1 189.1 mm to (24.6, 44.0), turned to 90 degrees
- moved R19 186.1 mm to (39.9, 112.5), turned to -90 degrees
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Connections:
- J3 pad 1: PB10 -> PA15
- J3 pad 2: PB13 -> PB4
- J3 pad 3: PB14 -> PB5
- J3 pad 4: PC13 -> PB9
- R24 pad 2: LED_MCU_SDA -> LED_MCU_SCL
- R33 pad 2: LED_MCU_SCL -> LED_MCU_SDA
- RGB1 pad 2: /RGB Array/SW1 -> /RGB Array/SW8
- RGB10 pad 2: /RGB Array/SW3 -> /RGB Array/SW6
- RGB11 pad 2: /RGB Array/SW4 -> /RGB Array/SW5
- RGB12 pad 2: /RGB Array/SW5 -> /RGB Array/SW4
- RGB13 pad 2: /RGB Array/SW6 -> /RGB Array/SW3
- RGB14 pad 2: /RGB Array/SW7 -> /RGB Array/SW2
- RGB15 pad 2: /RGB Array/SW1 -> /RGB Array/SW8
- RGB16 pad 2: /RGB Array/SW2 -> /RGB Array/SW7
- RGB17 pad 2: /RGB Array/SW3 -> /RGB Array/SW6
- RGB18 pad 2: /RGB Array/SW4 -> /RGB Array/SW5
- RGB19 pad 2: /RGB Array/SW5 -> /RGB Array/SW4
- RGB2 pad 2: /RGB Array/SW2 -> /RGB Array/SW7
- RGB20 pad 2: /RGB Array/SW6 -> /RGB Array/SW3
- RGB21 pad 2: /RGB Array/SW7 -> /RGB Array/SW2
- RGB22 pad 2: /RGB Array/SW1 -> /RGB Array/SW8
- RGB23 pad 2: /RGB Array/SW2 -> /RGB Array/SW7
- RGB24 pad 2: /RGB Array/SW3 -> /RGB Array/SW6
- RGB25 pad 2: /RGB Array/SW4 -> /RGB Array/SW5
- RGB26 pad 2: /RGB Array/SW5 -> /RGB Array/SW4
- RGB27 pad 2: /RGB Array/SW6 -> /RGB Array/SW3
- RGB28 pad 2: /RGB Array/SW7 -> /RGB Array/SW2
- RGB29 pad 2: /RGB Array/SW1 -> /RGB Array/SW8
- RGB3 pad 2: /RGB Array/SW3 -> /RGB Array/SW6
- RGB30 pad 2: /RGB Array/SW2 -> /RGB Array/SW7
- RGB31 pad 2: /RGB Array/SW3 -> /RGB Array/SW6
- RGB32 pad 2: /RGB Array/SW4 -> /RGB Array/SW5
- RGB33 pad 2: /RGB Array/SW5 -> /RGB Array/SW4
- RGB34 pad 2: /RGB Array/SW6 -> /RGB Array/SW3
- RGB35 pad 2: /RGB Array/SW7 -> /RGB Array/SW2
- RGB37 pad 2: /RGB Array/SW8 -> /RGB Array/SW1
- RGB4 pad 2: /RGB Array/SW4 -> /RGB Array/SW5
- RGB5 pad 2: /RGB Array/SW5 -> /RGB Array/SW4
- RGB6 pad 2: /RGB Array/SW6 -> /RGB Array/SW3
- RGB7 pad 2: /RGB Array/SW7 -> /RGB Array/SW2
- RGB8 pad 2: /RGB Array/SW1 -> /RGB Array/SW8
- RGB9 pad 2: /RGB Array/SW2 -> /RGB Array/SW7
- U6 pad 10: Col4 -> unconnected-(U6-PA2-Pad10)
- U6 pad 11: Col5 -> unconnected-(U6-PA3-Pad11)
- U6 pad 12: Col6 -> Row4
- U6 pad 13: Row2 -> Col5
- U6 pad 14: Row3 -> Col4
- U6 pad 15: Row4 -> Col3
- U6 pad 16: PB10 -> Col2
- U6 pad 17: unconnected-(U6-PB1-Pad17) -> Col1
- U6 pad 18: ThumbRow -> Col0
- U6 pad 2: PC13 -> ThumbRow
- U6 pad 22: unconnected-(U6-PB10-Pad22) -> Col6
- U6 pad 25: Row1 -> Row3
- U6 pad 26: Row0 -> Row2
- U6 pad 27: PB13 -> Row1
- U6 pad 28: PB14 -> Row0
- U6 pad 29: Col0 -> LED_MCU_SDB
- U6 pad 3: Col1 -> unconnected-(U6-PC14-Pad3)
- U6 pad 32: LED_MCU_SDB -> unconnected-(U6-PA10-Pad32)
- U6 pad 39: unconnected-(U6-PA15-Pad39) -> PA15
- U6 pad 41: unconnected-(U6-PB4-Pad41) -> PB4
- U6 pad 42: unconnected-(U6-PB5-Pad42) -> PB5
- U6 pad 46: unconnected-(U6-PB9-Pad46) -> PB9
- U6 pad 8: Col2 -> unconnected-(U6-PA0-Pad8)
- U6 pad 9: Col3 -> unconnected-(U6-PA1-Pad9)
Routing:
- net (no net): track 0.00 -> 154.8 mm
- net Row1: track 0.00 -> 151.9 mm
- net Row0: track 0.00 -> 149.7 mm
- net +3.3V: track 0.00 -> 114.6 mm
- net USB_MCU_D-: track 0.00 -> 111.1 mm
- net USB_MCU_D+: track 0.00 -> 111.1 mm
- net GND: track 0.00 -> 45.7 mm, vias 0 -> 33
- net RCC_OSC_IN: track 0.00 -> 7.49 mm
- net VBUS: track 0.00 -> 7.04 mm
- net USB_CONN_D+: track 0.00 -> 5.78 mm
- net USB_CONN_D-: track 0.00 -> 5.17 mm
- net RCC_OSC_OUT: track 0.00 -> 5.15 mm
- net Net-(USB1-CC1): track 0.00 -> 2.90 mm
- net Net-(USB1-CC2): track 0.00 -> 2.75 mm
- net /PWR_LED: track 0.00 -> 1.91 mm
- added copper zone on B.Cu, net +3.3V
- added copper zone on B.Cu, net +5V
- added copper zone on B.Cu, net GND
- added copper zone on F.Cu, net GND
- added copper zone on B.Cu, net VBUS
Other:
- outline, holes or cut-outs redrawn

Commit message: Save
Parts:
- moved H5 125.9 mm to (156.3, 29.7)
- moved USB2 114.1 mm to (139.2, 27.6), turned to 0 degrees
- moved U3 112.5 mm to (138.8, 34.8)
- moved R2 90.3 mm to (37.4, 34.1)
- moved C11 90.2 mm to (54.2, 36.1)
- moved R25 90.2 mm to (61.6, 35.0)
- moved U4 90.2 mm to (54.7, 31.0)
- moved USB1 90.2 mm to (35.5, 27.6)
- moved C10 90.2 mm to (47.9, 30.8)
- moved D39 90.2 mm to (58.8, 35.7)
- moved R1 90.2 mm to (33.3, 34.7)
- moved F1 90.2 mm to (44.4, 29.4)
- moved U2 90.2 mm to (35.3, 34.4)
- moved H2 41.8 mm to (4.78, 16.7)
- moved H6 41.8 mm to (-7.12, 16.7)
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Routing:
- net /RGB Array/G_RGB_ROW_0: track 0.00 -> 162.3 mm
- net /RGB Array/G_RGB_ROW_1: track 0.00 -> 159.8 mm
- net /RGB Array/G_RGB_ROW_2: track 0.00 -> 156.1 mm
- net Row3: track 0.00 -> 152.5 mm
- net /RGB Array/B_RGB_ROW_0: track 0.00 -> 152.4 mm
- net /RGB Array/B_RGB_ROW_2: track 0.00 -> 152.2 mm
- net /RGB Array/G_RGB_ROW_3: track 0.00 -> 152.0 mm, vias 0 -> 2
- net /RGB Array/B_RGB_ROW_1: track 0.00 -> 148.9 mm
- net /RGB Array/R_RGB_ROW_0: track 0.00 -> 148.1 mm, vias 0 -> 12
- net /RGB Array/B_RGB_ROW_3: track 0.00 -> 145.5 mm
- net /RGB Array/R_RGB_ROW_1: track 0.00 -> 143.6 mm, vias 0 -> 12
- net /RGB Array/R_RGB_ROW_2: track 0.00 -> 143.3 mm, vias 0 -> 12
- net /RGB Array/R_RGB_ROW_3: track 0.00 -> 140.8 mm, vias 0 -> 10
- net Row2: track 0.00 -> 136.4 mm
- net /RGB Array/G_RGB_ROW_4: track 0.00 -> 133.3 mm
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Other:
- outline, holes or cut-outs redrawn
