File: TheFalcon/PCB/TheFalcon[Left]/TheFalcon[Left].kicad_pcb (KiCad board)
At the start: 4 copper layers, 173.3 x 142.5 mm, 174 parts, among them IC1 IS31FL3729-QFLS4-TR, J1 Conn_01x01, J2 Conn_01x04_Pin, J3 Conn_01x01, J4 Conn_01x01, J5 Conn_01x01, J6 Conn_01x01, J7 Conn_01x01, SW1 SW_Push, SW2 SW_Push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

Commit message: Save
Parts:
- moved D36 44.0 mm to (118.0, 83.3)
- moved H1 44.0 mm to (118.3, 94.5)
- moved R23 44.0 mm to (10.9, 95.3)
- moved S13 44.0 mm to (105.8, 28.5)
- moved C11 44.0 mm to (28.3, -0.76)
- moved C12 44.0 mm to (66.2, 92.0)
- moved C7 44.0 mm to (97.3, 8.47)
- moved D24 44.0 mm to (56.6, 55.9)
- moved D27 44.0 mm to (113.7, 60.3)
- moved D29 44.0 mm to (18.3, 80.0)
- moved D3 44.0 mm to (56.4, 2.57)
- moved D30 44.0 mm to (37.5, 80.1)
- moved D38 44.0 mm to (148.5, 97.0)
- moved H4 44.0 mm to (139.7, 100.8)
- moved J1 44.0 mm to (113.7, 10.6)
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
Commit message: Save
Parts:
- moved C11 41.0 mm to (52.5, 32.3)
- moved C12 41.0 mm to (90.4, 125.0)
- moved C14 41.0 mm to (96.4, 130.1)
- moved C5 41.0 mm to (119.4, 36.5)
- moved D17 41.0 mm to (80.4, 70.0)
- moved D20 41.0 mm to (138.2, 74.4)
- moved D21 41.0 mm to (157.3, 74.2)
- moved D30 41.0 mm to (61.7, 113.2)
- moved H1 41.0 mm to (142.6, 127.6)
- moved H3 41.0 mm to (138.3, 60.0)
- moved R14 41.0 mm to (28.2, 66.7)
- moved R21 41.0 mm to (72.9, 128.3)
- moved R24 41.0 mm to (101.9, 35.2)
- moved RGB13 41.0 mm to (130.7, 66.7)
- moved RGB14 41.0 mm to (149.7, 66.7)
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Routing:
- net Net-(D7-A): track 4.55 -> 3.55 mm

Commit message: Save
Connections:
- H1 pad 1: GND -> unconnected-(H1-Pad1)
- H2 pad 1: GND -> unconnected-(H2-Pad1)
- H3 pad 1: GND -> unconnected-(H3-Pad1)
- H4 pad 1: GND -> unconnected-(H4-Pad1)
- H5 pad 1: GND -> unconnected-(H5-Pad1)
- H6 pad 1: GND -> unconnected-(H6-Pad1)
Routing:
- net unconnected-(USB1-SHIELD-PadS1)_1: track 17.0 -> 0.00 mm
- net unconnected-(USB2-SHIELD-PadS1)_2: track 17.0 -> 0.00 mm
Changed lines of the file:
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@@
 	(net 134 "unconnected-(U6-PB11-Pad25)")
 	(net 135 "unconnected-(U6-PB5-Pad42)")
+	(net 136 "unconnected-(H1-Pad1)")
+	(net 137 "unconnected-(H2-Pad1)")
+	(net 138 "unconnected-(H3-Pad1)")
+	(net 139 "unconnected-(H4-Pad1)")
+	(net 140 "unconnected-(H5-Pad1)")
+	(net 141 "unconnected-(H6-Pad1)")
+	(net 142 "unconnected-(USB1-SHIELD-PadS1)_1")
+	(net 143 "unconnected-(USB1-SHIELD-PadS1)_2")
+	(net 144 "unconnected-(USB1-SHIELD-PadS1)_3")
+	(net 145 "unconnected-(USB2-SHIELD-PadS1)_1")
+	(net 146 "unconnected-(USB2-SHIELD-PadS1)_2")
+	(net 147 "unconnected-(USB2-SHIELD-PadS1)_3")
 	(footprint "SamacSys_Parts:T36K3BGR05D000121U1930_MODEL_INVERTED"
 		(layer "F.Cu")
@@
 			(layers "*.Cu" "*.Mask")
 			(remove_unused_layers no)
-			(net 1 "GND")
+			(net 137 "unconnected-(H2-Pad1)")
 			(pinfunction "1")
-			(pintype "input")
+			(pintype "input+no_connect")
 			(zone_connect 2)
 		)
@@
 			(layers "*.Cu" "*.Mask")
 			(remove_unused_layers no)
-			(net 116 "unconnected-(USB1-SHIELD-PadS1)")
+			(net 144 "unconnected-(USB1-SHIELD-PadS1)_3")
 			(pinfunction "SHIELD")
 			(pintype "passive+no_connect")
@@
 			(layers "*.Cu" "*.Mask")
 			(remove_unused_layers no)
-			(net 116 "unconnected-(USB1-SHIELD-PadS1)")
+			(net 143 "unconnected-(USB1-SHIELD-PadS1)_2")
 			(pinfunction "SHIELD")
 			(pintype "passive+no_connect")
@@
 			(layers "*.Cu" "*.Mask")
 			(remove_unused_layers no)
-			(net 116 "unconnected-(USB1-SHIELD-PadS1)")
+			(net 142 "unconnected-(USB1-SHIELD-PadS1)_1")
 			(pinfunction "SHIELD")
 			(pintype "passive+no_connect")
@@
 			(layers "*.Cu" "*.Mask")
 			(remove_unused_layers no)
-			(net 1 "GND")
+			(net 141 "unconnected-(H6-Pad1)")
 			(pinfunction "1")
-			(pintype "input")
+			(pintype "input+no_connect")
 			(zone_connect 2)
 		)
@@
 			(layers "*.Cu" "*.Mask")
 			(remove_unused_layers no)
-			(net 119 "unconnected-(USB2-SHIELD-PadS1)")
+			(net 147 "unconnected-(USB2-SHIELD-PadS1)_3")
 			(pinfunction "SHIELD")
 			(pintype "passive+no_connect")
@@
 			(layers "*.Cu" "*.Mask")
 			(remove_unused_layers no)
-			(net 119 "unconnected-(USB2-SHIELD-PadS1)")
+			(net 145 "unconnected-(USB2-SHIELD-PadS1)_1")
 			(pinfunction "SHIELD")
 			(pintype "passive+no_connect")
@@
 			(layers "*.Cu" "*.Mask")
 			(remove_unused_layers no)
-			(net 119 "unconnected-(USB2-SHIELD-PadS1)")
+			(net 146 "unconnected-(USB2-SHIELD-PadS1)_2")
 			(pinfunction "SHIELD")
 			(pintype "passive+no_connect")
@@
 			(layers "*.Cu" "*.Mask")
 			(remove_unused_layers no)
-			(net 1 "GND")
+			(net 140 "unconnected-(H5-Pad1)")
 			(pinfunction "1")
-			(pintype "input")
+			(pintype "input+no_connect")
 			(zone_connect 2)
 		)
@@
 			(layers "*.Cu" "*.Mask")
 			(remove_unused_layers no)
-			(net 1 "GND")
+			(net 139 "unconnected-(H4-Pad1)")
 			(pinfunction "1")
-			(pintype "input")
+			(pintype "input+no_connect")
 			(zone_connect 2)
 		)
@@
 			(layers "*.Cu" "*.Mask")
 			(remove_unused_layers no)
-			(net 1 "GND")
+			(net 136 "unconnected-(H1-Pad1)")
 			(pinfunction "1")
-			(pintype "input")
+			(pintype "input+no_connect")
 			(zone_connect 2)
 		)
@@
 			(layers "*.Cu" "*.Mask")
 			(remove_unused_layers no)
-			(net 1 "GND")
+			(net 138 "unconnected-(H3-Pad1)")
 			(pinfunction "1")
-			(pintype "input")
+			(pintype "input+no_connect")
 			(zone_connect 2)
 		)
@@
 	)
 	(segment
-		(start 39.06 25.9825)
-		(end 39.06 21.7825)
-		(width 0.2)
-		(layer "F.Cu")
-		(net 116)
-	)
-	(segment
-		(start 30.42 21.7825)
-		(end 30.42 25.9825)
-		(width 0.2)
-		(layer "F.Cu")
-		(net 116)
-	)
-	(segment
-		(start 39.06 21.7825)
-		(end 30.42 21.7825)
-		(width 0.2)
-		(layer "F.Cu")
-		(net 116)
-	)
-	(segment
-		(start 160.875 23.73)
-		(end 156.675 23.73)
-		(width 0.2)
-		(layer "F.Cu")
-		(net 119)
-	)
-	(segment
-		(start 156.675 32.37)
-		(end 160.875 32.37)
-		(width 0.2)
-		(layer "F.Cu")
-		(net 119)
-	)
-	(segment
-		(start 160.875 32.37)
-		(end 160.875 23.73)
-		(width 0.2)
-		(layer "F.Cu")
-		(net 119)
-	)
-	(segment

Commit message: save
Parts:
- removed H1, H2, H3, H4, H5, H6: MountingHole_Pad, MountingHole:MountingHole_2.2mm_M2_Pad
Routing:
- net +5V: track 257.6 -> 259.9 mm
- net SYS_JTAG_TRACE: track 146.8 -> 144.7 mm
- net SYS_JTAG_SWCLK: track 144.4 -> 142.7 mm
- net SYS_JTAG_SWDIO: track 136.8 -> 135.4 mm
- net VBUS: track 130.2 -> 131.5 mm
- net /RGB Array/SW2: track 194.4 -> 195.2 mm
- net Col6: track 150.5 -> 151.2 mm
- net /RGB Array/R_RGB_ROW_3: track 155.8 -> 155.1 mm
- net GND: vias 135 -> 134
Other:
- outline, holes or cut-outs redrawn
- board text added: "SPACER"
