File: TheFalcon/PCB/TheFalcon[Left]/TheFalcon[Left].kicad_sch (KiCad schematic)
At the start: 42 parts, among them J2 Conn_01x04_Pin, J3 Conn_01x04_Pin, J5 Conn_01x01, J6 Conn_01x01, SW1 SW_Push, SW2 SW_Push, U2 USBLC6-2P6, U3 USBLC6-2P6, U4 AMS1117-3.3, U6 STM32G431CBTx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

Commit message: Cleaning up
I have all connections, just cleaning up
Parts:
- removed J3: Conn_01x04_Pin, Connector_Wire:SolderWire-1sqmm_1x04_P5.4mm_D1.4mm_OD2.7mm, symbol Connector:Conn_01x04_Pin
- added J1, J3, J4, J7: Conn_01x01, Connector_Wire:SolderWire-0.1sqmm_1x01_D0.4mm_OD1mm, symbol Connector_Generic:Conn_01x01
Connections:
- net PA15: now also J1.1 (Pin_1)
- net PB4: now also J3.1 (Pin_1)
- net PB9: now also U6.16 (PB0), J7.1 (Pin_1); no longer U6.46 (PB9)
- net PB5: no longer names the net of U6.42 (PB5)
- no-connect marks 15 -> 17

Commit message: Save
Connections:
- net GND: no longer H1.1, H2.1, H3.1, H4.1, H5.1, H6.1
- no-connect marks 17 -> 23
Changed lines of the file:
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@@
 	)
 	(junction
-		(at 147.32 45.72)
-		(diameter 0)
-		(color 0 0 0 0)
-	)
-	(junction
 		(at 63.5 35.56)
 		(diameter 0)
@@
 	)
 	(junction
-		(at 147.32 30.48)
-		(diameter 0)
-		(color 0 0 0 0)
-	)
-	(junction
 		(at 95.25 68.58)
 		(diameter 0)
@@
 	)
 	(junction
-		(at 147.32 40.64)
-		(diameter 0)
-		(color 0 0 0 0)
-	)
-	(junction
 		(at 105.41 22.86)
 		(diameter 0)
@@
 	)
 	(junction
-		(at 147.32 25.4)
-		(diameter 0)
-		(color 0 0 0 0)
-	)
-	(junction
 		(at 95.25 33.02)
 		(diameter 0)
@@
 	)
 	(junction
-		(at 147.32 35.56)
-		(diameter 0)
-		(color 0 0 0 0)
-	)
-	(junction
 		(at 30.48 182.88)
 		(diameter 0)
@@
 	)
 	(no_connect
+		(at 147.32 25.4)
+	)
+	(no_connect
 		(at 86.36 63.5)
 	)
@@
 	)
 	(no_connect
+		(at 147.32 35.56)
+	)
+	(no_connect
 		(at 45.72 78.74)
 	)
@@
 	)
 	(no_connect
+		(at 147.32 30.48)
+	)
+	(no_connect
 		(at 45.72 101.6)
 	)
@@
 	)
 	(no_connect
+		(at 147.32 20.32)
+	)
+	(no_connect
+		(at 147.32 45.72)
+	)
+	(no_connect
 		(at 96.52 172.72)
 	)
 	(no_connect
+		(at 147.32 40.64)
+	)
+	(no_connect
 		(at 96.52 175.26)
 	)
@@
 	(wire
 		(pts
-			(xy 147.32 35.56) (xy 147.32 40.64)
-		)
-		(stroke
-			(width 0)
-			(type default)
-		)
-	)
-	(wire
-		(pts
 			(xy 57.15 22.86) (xy 57.15 24.13)
 		)
@@
 	(wire
 		(pts
-			(xy 147.32 20.32) (xy 147.32 25.4)
-		)
-		(stroke
-			(width 0)
-			(type default)
-		)
-	)
-	(wire
-		(pts
 			(xy 45.72 55.88) (xy 48.26 55.88)
 		)
@@
 	(wire
 		(pts
-			(xy 147.32 40.64) (xy 147.32 45.72)
-		)
-		(stroke
-			(width 0)
-			(type default)
-		)
-	)
-	(wire
-		(pts
-			(xy 147.32 30.48) (xy 147.32 35.56)
-		)
-		(stroke
-			(width 0)
-			(type default)
-		)
-	)
-	(wire
-		(pts
 			(xy 222.25 134.62) (xy 219.71 134.62)
 		)
@@
 	(wire
 		(pts
-			(xy 147.32 45.72) (xy 147.32 48.26)
-		)
-		(stroke
-			(width 0)
-			(type default)
-		)
-	)
-	(wire
-		(pts
 			(xy 266.7 134.62) (xy 266.7 137.16)
 		)
@@
 	(wire
 		(pts
-			(xy 147.32 25.4) (xy 147.32 30.48)
-		)
-		(stroke
-			(width 0)
-			(type default)
-		)
-	)
-	(wire
-		(pts
 			(xy 45.72 58.42) (xy 48.26 58.42)
 		)
@@
 					(unit 1)
 				)
-			)
-		)
-	)
-	(symbol
-		(lib_id "power:GND")
-		(at 147.32 48.26 0)
-		(unit 1)
-		(exclude_from_sim no)
-		(in_bom yes)
-		(on_board yes)
-		(dnp no)
-		(property "Reference" "#PWR036"
-			(at 147.32 54.61 0)
-			(effects
-				(font
-					(size 1.27 1.27)
-				)
-				(hide yes)
-			)
-		)
-		(property "Value" "GND"
-			(at 147.32 53.34 0)
-			(effects
-				(font
-					(size 1.27 1.27)
-				)
-			)
-		)
-		(property "Footprint" ""
-			(at 147.32 48.26 0)
-			(effects
-				(font
-					(size 1.27 1.27)
-				)
-				(hide yes)
-			)
-		)
-		(property "Datasheet" ""
-			(at 147.32 48.26 0)
-			(effects
-				(font
-					(size 1.27 1.27)
-				)
-				(hide yes)
-			)
-		)
-		(property "Description" "Power symbol creates a global label with name \"GND\" , ground"
-			(at 147.32 48.26 0)
-			(effects
-				(font
-					(size 1.27 1.27)
-				)
-				(hide yes)
-			)
-		)
-		(pin "1"
-		)
-		(instances
-			(project "TheFalcon[Left]"
-				(path "/7314d873-34d2-434b-a863-40da9c12efca"
-					(reference "#PWR036")
-					(unit 1)
-				)

Commit message: save
Parts:
- removed H1, H2, H3, H4, H5, H6: MountingHole_Pad, MountingHole:MountingHole_2.2mm_M2_Pad, symbol Mechanical:MountingHole_Pad
Connections:
- no-connect marks 23 -> 17

Commit message: Files ready for production
Going to panelise seperate files to reduce PCBA cost
Parts:
- C1: LCSC Part Number (none) -> C1713
- C10, C11: LCSC Part Number (none) -> C1859
- C15, C16: LCSC Part Number (none) -> C1545
- C17, C7: LCSC Part Number (none) -> C1592
- C2, C3, C4, C5, C8, C9: LCSC Part Number (none) -> C1525
- C6: LCSC Part Number (none) -> C1524
- D39: LCSC Part Number (none) -> C84260
- F1: LCSC Part Number (none) -> C135336
- R1, R2, R3, R4: value 5.1k -> 5k1; LCSC Part Number (none) -> C23067
- R24, R33: LCSC Part Number (none) -> C23162
- R25: LCSC Part Number (none) -> C22843
- SW1, SW2: footprint Button_Switch_SMD:SW_SPST_B3U-1000P -> CustomSPDTButton:SPDT_Switch_KiCad_BasicComponent; LCSC Part Number (none) -> C231329
- U2: LCSC Part Number (none) -> C29780639; Link https://jlcpcb.com/partdetail/31512546-USBLC6_2P6_UMW/C2978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 -> (none)
- U3: LCSC Part Number (none) -> C29780639
- U4: LCSC Part Number (none) -> C6186; Link https://jlcpcb.com/partdetail/Advanced_MonolithicSystems-AM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 -> (none)
- U6: LCSC Part Number (none) -> C529355
- USB1, USB2: LCSC Part Number (none) -> C2988369; Link https://jlcpcb.com/partdetail/gswitch-GT_USB7010ASV/C2988369 -> (none)
- Y1: Height 0.8 -> (none); LCSC Part Number (none) -> C12668; Link1 https://jlcpcb.com/partdetail/Yxc_CrystalOscillators-X32251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 -> (none); Link2 https://za.rs-online.com/web/p/crystal-units/1712765?cm_mmc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 -> (none); Manufacturer_Name Yangxing Tech -> (none); Manufacturer_Part_Number X322516MOB4SI -> (none)
