File: TheFalcon/PCB/TheFalcon[Left]/_autosave-RGBArray.kicad_sch (KiCad schematic)
At the start: 57 parts, among them IC1 IS31FL3729-QFLS4-TR

Commit message: Save
Connections:
- net +5V: no longer IC1.28 (AD)
- net GND: now also IC1.28 (AD)
Other:
- moved on the sheet: C12, C13, C14, IC1, R10, R11, R12, R13, R14, R15, R16, R17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
