File: TheFalcon/PCB/TheFalcon[Left]/KeyMatrix.kicad_sch (KiCad schematic)
At the start: 76 parts

Commit message: Save
Parts:
- removed D34, D35: Diode, Diode_SMD:D_SOD-123, symbol ScottoKeebs:Placeholder_Diode
- removed S34, S35: Keyswitch, Gateron_KS33_Hotswap:Gateron-KS33-Hotswap-1U, symbol ScottoKeebs:Placeholder_Keyswitch
- S1, S10, S11, S12, S13, S14, S15, S16, S17, S18, S19, S2, S20, S21, S22, S23, S24, S25, S26, S27, S28, S29, S3, S30, S31, S32, S33, S4, S5, S6, S7, S8, S9: footprint Gateron_KS33_Hotswap:Gateron-KS33-Hotswap-1U -> Gateron_KS33_Hotswap:Gateron-KS33-Hotswap-1U_Model
- S34: renamed from S36; footprint Gateron_KS33_Hotswap:Gateron-KS33-Hotswap-1U -> Gateron_KS33_Hotswap:Gateron-KS33-Hotswap-1U_Model
- renumbered S37 to S35, S38 to S36

Commit message: Save
Parts:
- S1, S10, S11, S12, S13, S14, S15, S16, S17, S18, S19, S2, S20, S21, S22, S23, S24, S25, S26, S27, S28, S29, S3, S30, S31, S32, S33, S34, S4, S5, S6, S7, S8, S9: footprint Gateron_KS33_Hotswap:Gateron-KS33-Hotswap-1U_Model -> Gateron_KS33_Hotswap:Gateron-KS33-Hotswap-1U
Changed lines of the file:
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@@
 			)
 		)
-		(property "Footprint" "Gateron_KS33_Hotswap:Gateron-KS33-Hotswap-1U_Model"
+		(property "Footprint" "Gateron_KS33_Hotswap:Gateron-KS33-Hotswap-1U"
 			(at 38.1 114.3 0)
 			(effects
@@
 			)
 		)
-		(property "Footprint" "Gateron_KS33_Hotswap:Gateron-KS33-Hotswap-1U_Model"
+		(property "Footprint" "Gateron_KS33_Hotswap:Gateron-KS33-Hotswap-1U"
 			(at 76.2 114.3 0)
 			(effects
@@
 			)
 		)
-		(property "Footprint" "Gateron_KS33_Hotswap:Gateron-KS33-Hotswap-1U_Model"
+		(property "Footprint" "Gateron_KS33_Hotswap:Gateron-KS33-Hotswap-1U"
 			(at 88.9 63.5 0)
 			(effects
@@
 			)
 		)
-		(property "Footprint" "Gateron_KS33_Hotswap:Gateron-KS33-Hotswap-1U_Model"
+		(property "Footprint" "Gateron_KS33_Hotswap:Gateron-KS33-Hotswap-1U"
 			(at 25.4 139.7 0)
 			(effects
@@
 			)
 		)
-		(property "Footprint" "Gateron_KS33_Hotswap:Gateron-KS33-Hotswap-1U_Model"
+		(property "Footprint" "Gateron_KS33_Hotswap:Gateron-KS33-Hotswap-1U"
 			(at 25.4 38.1 0)
 			(effects
@@
 			)
 		)
-		(property "Footprint" "Gateron_KS33_Hotswap:Gateron-KS33-Hotswap-1U_Model"
+		(property "Footprint" "Gateron_KS33_Hotswap:Gateron-KS33-Hotswap-1U"
 			(at 101.6 114.3 0)
 			(effects
@@
 			)
 		)
-		(property "Footprint" "Gateron_KS33_Hotswap:Gateron-KS33-Hotswap-1U_Model"
+		(property "Footprint" "Gateron_KS33_Hotswap:Gateron-KS33-Hotswap-1U"
 			(at 63.5 139.7 0)
 			(effects
@@
 			)
 		)
-		(property "Footprint" "Gateron_KS33_Hotswap:Gateron-KS33-Hotswap-1U_Model"
+		(property "Footprint" "Gateron_KS33_Hotswap:Gateron-KS33-Hotswap-1U"
 			(at 76.2 88.9 0)
 			(effects
@@
 			)
 		)
-		(property "Footprint" "Gateron_KS33_Hotswap:Gateron-KS33-Hotswap-1U_Model"
+		(property "Footprint" "Gateron_KS33_Hotswap:Gateron-KS33-Hotswap-1U"
 			(at 25.4 88.9 0)
 			(effects
@@
 			)
 		)
-		(property "Footprint" "Gateron_KS33_Hotswap:Gateron-KS33-Hotswap-1U_Model"
+		(property "Footprint" "Gateron_KS33_Hotswap:Gateron-KS33-Hotswap-1U"
 			(at 76.2 139.7 0)
 			(effects
@@
 			)
 		)
-		(property "Footprint" "Gateron_KS33_Hotswap:Gateron-KS33-Hotswap-1U_Model"
+		(property "Footprint" "Gateron_KS33_Hotswap:Gateron-KS33-Hotswap-1U"
 			(at 25.4 114.3 0)
 			(effects
@@
 			)
 		)
-		(property "Footprint" "Gateron_KS33_Hotswap:Gateron-KS33-Hotswap-1U_Model"
+		(property "Footprint" "Gateron_KS33_Hotswap:Gateron-KS33-Hotswap-1U"
 			(at 38.1 139.7 0)
 			(effects
@@
 			)
 		)
-		(property "Footprint" "Gateron_KS33_Hotswap:Gateron-KS33-Hotswap-1U_Model"
+		(property "Footprint" "Gateron_KS33_Hotswap:Gateron-KS33-Hotswap-1U"
 			(at 63.5 63.5 0)
 			(effects
@@
 			)
 		)
-		(property "Footprint" "Gateron_KS33_Hotswap:Gateron-KS33-Hotswap-1U_Model"
+		(property "Footprint" "Gateron_KS33_Hotswap:Gateron-KS33-Hotswap-1U"
 			(at 88.9 88.9 0)
 			(effects
@@
 			)
 		)
-		(property "Footprint" "Gateron_KS33_Hotswap:Gateron-KS33-Hotswap-1U_Model"
+		(property "Footprint" "Gateron_KS33_Hotswap:Gateron-KS33-Hotswap-1U"
 			(at 88.9 38.1 0)
 			(effects
@@
 			)
 		)
-		(property "Footprint" "Gateron_KS33_Hotswap:Gateron-KS33-Hotswap-1U_Model"
+		(property "Footprint" "Gateron_KS33_Hotswap:Gateron-KS33-Hotswap-1U"
 			(at 101.6 38.1 0)
 			(effects
@@
 			)
 		)
-		(property "Footprint" "Gateron_KS33_Hotswap:Gateron-KS33-Hotswap-1U_Model"
+		(property "Footprint" "Gateron_KS33_Hotswap:Gateron-KS33-Hotswap-1U"
 			(at 63.5 88.9 0)
 			(effects
@@
 			)
 		)
-		(property "Footprint" "Gateron_KS33_Hotswap:Gateron-KS33-Hotswap-1U_Model"
+		(property "Footprint" "Gateron_KS33_Hotswap:Gateron-KS33-Hotswap-1U"
 			(at 76.2 63.5 0)
 			(effects
@@
 			)
 		)
-		(property "Footprint" "Gateron_KS33_Hotswap:Gateron-KS33-Hotswap-1U_Model"
+		(property "Footprint" "Gateron_KS33_Hotswap:Gateron-KS33-Hotswap-1U"
 			(at 50.8 63.5 0)
 			(effects
@@
 			)
 		)
-		(property "Footprint" "Gateron_KS33_Hotswap:Gateron-KS33-Hotswap-1U_Model"
+		(property "Footprint" "Gateron_KS33_Hotswap:Gateron-KS33-Hotswap-1U"
 			(at 63.5 38.1 0)
 			(effects
@@
 			)
 		)
-		(property "Footprint" "Gateron_KS33_Hotswap:Gateron-KS33-Hotswap-1U_Model"
+		(property "Footprint" "Gateron_KS33_Hotswap:Gateron-KS33-Hotswap-1U"
 			(at 50.8 38.1 0)
 			(effects
@@
 			)
 		)
-		(property "Footprint" "Gateron_KS33_Hotswap:Gateron-KS33-Hotswap-1U_Model"
+		(property "Footprint" "Gateron_KS33_Hotswap:Gateron-KS33-Hotswap-1U"
 			(at 101.6 88.9 0)
 			(effects
@@
 			)
 		)
-		(property "Footprint" "Gateron_KS33_Hotswap:Gateron-KS33-Hotswap-1U_Model"
+		(property "Footprint" "Gateron_KS33_Hotswap:Gateron-KS33-Hotswap-1U"
 			(at 88.9 114.3 0)
 			(effects
@@
 			)
 		)
-		(property "Footprint" "Gateron_KS33_Hotswap:Gateron-KS33-Hotswap-1U_Model"
+		(property "Footprint" "Gateron_KS33_Hotswap:Gateron-KS33-Hotswap-1U"
 			(at 38.1 38.1 0)
 			(effects
@@
 			)
 		)
-		(property "Footprint" "Gateron_KS33_Hotswap:Gateron-KS33-Hotswap-1U_Model"
+		(property "Footprint" "Gateron_KS33_Hotswap:Gateron-KS33-Hotswap-1U"
 			(at 38.1 88.9 0)
 			(effects
@@
 			)
 		)
-		(property "Footprint" "Gateron_KS33_Hotswap:Gateron-KS33-Hotswap-1U_Model"
+		(property "Footprint" "Gateron_KS33_Hotswap:Gateron-KS33-Hotswap-1U"
 			(at 76.2 165.1 0)
 			(effects
@@
 			)
 		)
-		(property "Footprint" "Gateron_KS33_Hotswap:Gateron-KS33-Hotswap-1U_Model"
+		(property "Footprint" "Gateron_KS33_Hotswap:Gateron-KS33-Hotswap-1U"
 			(at 38.1 63.5 0)
 			(effects
@@
 			)
 		)
-		(property "Footprint" "Gateron_KS33_Hotswap:Gateron-KS33-Hotswap-1U_Model"
+		(property "Footprint" "Gateron_KS33_Hotswap:Gateron-KS33-Hotswap-1U"
 			(at 101.6 63.5 0)
 			(effects
@@
 			)
 		)
-		(property "Footprint" "Gateron_KS33_Hotswap:Gateron-KS33-Hotswap-1U_Model"
+		(property "Footprint" "Gateron_KS33_Hotswap:Gateron-KS33-Hotswap-1U"
 			(at 76.2 38.1 0)
 			(effects
@@
 			)
 		)
-		(property "Footprint" "Gateron_KS33_Hotswap:Gateron-KS33-Hotswap-1U_Model"
+		(property "Footprint" "Gateron_KS33_Hotswap:Gateron-KS33-Hotswap-1U"
 			(at 25.4 63.5 0)
 			(effects
@@
 			)
 		)
-		(property "Footprint" "Gateron_KS33_Hotswap:Gateron-KS33-Hotswap-1U_Model"
+		(property "Footprint" "Gateron_KS33_Hotswap:Gateron-KS33-Hotswap-1U"
 			(at 50.8 88.9 0)
 			(effects
@@
 			)
 		)
-		(property "Footprint" "Gateron_KS33_Hotswap:Gateron-KS33-Hotswap-1U_Model"
+		(property "Footprint" "Gateron_KS33_Hotswap:Gateron-KS33-Hotswap-1U"
 			(at 50.8 114.3 0)
 			(effects
@@
 			)
 		)
-		(property "Footprint" "Gateron_KS33_Hotswap:Gateron-KS33-Hotswap-1U_Model"
+		(property "Footprint" "Gateron_KS33_Hotswap:Gateron-KS33-Hotswap-1U"
 			(at 63.5 114.3 0)
 			(effects
@@
 			)
 		)
-		(property "Footprint" "Gateron_KS33_Hotswap:Gateron-KS33-Hotswap-1U_Model"
+		(property "Footprint" "Gateron_KS33_Hotswap:Gateron-KS33-Hotswap-1U"
 			(at 50.8 139.7 0)
 			(effects

Commit message: Save
Parts:
- S1, S10, S11, S12, S13, S14, S15, S16, S17, S18, S19, S2, S20, S21, S22, S23, S24, S25, S26, S27, S28, S29, S3, S30, S31, S32, S33, S34, S4, S5, S6, S7, S8, S9: footprint Gateron_KS33_Hotswap:Gateron-KS33-Hotswap-1U -> MX_KS33:MX_KS33-Solderable-1U
- S35, S36: footprint Gateron_KS33_Hotswap:Gateron-KS33-Hotswap-1.5U -> MX_KS33:MX_KS33-Solderable-1.5U
Changed lines of the file:
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@@
 			)
 		)
-		(property "Footprint" "Gateron_KS33_Hotswap:Gateron-KS33-Hotswap-1U"
+		(property "Footprint" "MX_KS33:MX_KS33-Solderable-1U"
 			(at 38.1 114.3 0)
 			(effects
@@
 			)
 		)
-		(property "Footprint" "Gateron_KS33_Hotswap:Gateron-KS33-Hotswap-1U"
+		(property "Footprint" "MX_KS33:MX_KS33-Solderable-1U"
 			(at 76.2 114.3 0)
 			(effects
@@
 			)
 		)
-		(property "Footprint" "Gateron_KS33_Hotswap:Gateron-KS33-Hotswap-1U"
+		(property "Footprint" "MX_KS33:MX_KS33-Solderable-1U"
 			(at 88.9 63.5 0)
 			(effects
@@
 			)
 		)
-		(property "Footprint" "Gateron_KS33_Hotswap:Gateron-KS33-Hotswap-1U"
+		(property "Footprint" "MX_KS33:MX_KS33-Solderable-1U"
 			(at 25.4 139.7 0)
 			(effects
@@
 			)
 		)
-		(property "Footprint" "Gateron_KS33_Hotswap:Gateron-KS33-Hotswap-1U"
+		(property "Footprint" "MX_KS33:MX_KS33-Solderable-1U"
 			(at 25.4 38.1 0)
 			(effects
@@
 			)
 		)
-		(property "Footprint" "Gateron_KS33_Hotswap:Gateron-KS33-Hotswap-1U"
+		(property "Footprint" "MX_KS33:MX_KS33-Solderable-1U"
 			(at 101.6 114.3 0)
 			(effects
@@
 			)
 		)
-		(property "Footprint" "Gateron_KS33_Hotswap:Gateron-KS33-Hotswap-1U"
+		(property "Footprint" "MX_KS33:MX_KS33-Solderable-1U"
 			(at 63.5 139.7 0)
 			(effects
@@
 			)
 		)
-		(property "Footprint" "Gateron_KS33_Hotswap:Gateron-KS33-Hotswap-1U"
+		(property "Footprint" "MX_KS33:MX_KS33-Solderable-1U"
 			(at 76.2 88.9 0)
 			(effects
@@
 			)
 		)
-		(property "Footprint" "Gateron_KS33_Hotswap:Gateron-KS33-Hotswap-1U"
+		(property "Footprint" "MX_KS33:MX_KS33-Solderable-1U"
 			(at 25.4 88.9 0)
 			(effects
@@
 			)
 		)
-		(property "Footprint" "Gateron_KS33_Hotswap:Gateron-KS33-Hotswap-1U"
+		(property "Footprint" "MX_KS33:MX_KS33-Solderable-1U"
 			(at 76.2 139.7 0)
 			(effects
@@
 			)
 		)
-		(property "Footprint" "Gateron_KS33_Hotswap:Gateron-KS33-Hotswap-1.5U"
+		(property "Footprint" "MX_KS33:MX_KS33-Solderable-1.5U"
 			(at 88.9 165.1 0)
 			(effects
@@
 			)
 		)
-		(property "Footprint" "Gateron_KS33_Hotswap:Gateron-KS33-Hotswap-1U"
+		(property "Footprint" "MX_KS33:MX_KS33-Solderable-1U"
 			(at 25.4 114.3 0)
 			(effects
@@
 			)
 		)
-		(property "Footprint" "Gateron_KS33_Hotswap:Gateron-KS33-Hotswap-1U"
+		(property "Footprint" "MX_KS33:MX_KS33-Solderable-1U"
 			(at 38.1 139.7 0)
 			(effects
@@
 			)
 		)
-		(property "Footprint" "Gateron_KS33_Hotswap:Gateron-KS33-Hotswap-1U"
+		(property "Footprint" "MX_KS33:MX_KS33-Solderable-1U"
 			(at 63.5 63.5 0)
 			(effects
@@
 			)
 		)
-		(property "Footprint" "Gateron_KS33_Hotswap:Gateron-KS33-Hotswap-1U"
+		(property "Footprint" "MX_KS33:MX_KS33-Solderable-1U"
 			(at 88.9 88.9 0)
 			(effects
@@
 			)
 		)
-		(property "Footprint" "Gateron_KS33_Hotswap:Gateron-KS33-Hotswap-1U"
+		(property "Footprint" "MX_KS33:MX_KS33-Solderable-1U"
 			(at 88.9 38.1 0)
 			(effects
@@
 			)
 		)
-		(property "Footprint" "Gateron_KS33_Hotswap:Gateron-KS33-Hotswap-1U"
+		(property "Footprint" "MX_KS33:MX_KS33-Solderable-1U"
 			(at 101.6 38.1 0)
 			(effects
@@
 			)
 		)
-		(property "Footprint" "Gateron_KS33_Hotswap:Gateron-KS33-Hotswap-1U"
+		(property "Footprint" "MX_KS33:MX_KS33-Solderable-1U"
 			(at 63.5 88.9 0)
 			(effects
@@
 			)
 		)
-		(property "Footprint" "Gateron_KS33_Hotswap:Gateron-KS33-Hotswap-1U"
+		(property "Footprint" "MX_KS33:MX_KS33-Solderable-1U"
 			(at 76.2 63.5 0)
 			(effects
@@
 			)
 		)
-		(property "Footprint" "Gateron_KS33_Hotswap:Gateron-KS33-Hotswap-1U"
+		(property "Footprint" "MX_KS33:MX_KS33-Solderable-1U"
 			(at 50.8 63.5 0)
 			(effects
@@
 			)
 		)
-		(property "Footprint" "Gateron_KS33_Hotswap:Gateron-KS33-Hotswap-1U"
+		(property "Footprint" "MX_KS33:MX_KS33-Solderable-1U"
 			(at 63.5 38.1 0)
 			(effects
@@
 			)
 		)
-		(property "Footprint" "Gateron_KS33_Hotswap:Gateron-KS33-Hotswap-1U"
+		(property "Footprint" "MX_KS33:MX_KS33-Solderable-1U"
 			(at 50.8 38.1 0)
 			(effects
@@
 			)
 		)
-		(property "Footprint" "Gateron_KS33_Hotswap:Gateron-KS33-Hotswap-1U"
+		(property "Footprint" "MX_KS33:MX_KS33-Solderable-1U"
 			(at 101.6 88.9 0)
 			(effects
@@
 			)
 		)
-		(property "Footprint" "Gateron_KS33_Hotswap:Gateron-KS33-Hotswap-1U"
+		(property "Footprint" "MX_KS33:MX_KS33-Solderable-1U"
 			(at 88.9 114.3 0)
 			(effects
@@
 			)
 		)
-		(property "Footprint" "Gateron_KS33_Hotswap:Gateron-KS33-Hotswap-1U"
+		(property "Footprint" "MX_KS33:MX_KS33-Solderable-1U"
 			(at 38.1 38.1 0)
 			(effects
@@
 			)
 		)
-		(property "Footprint" "Gateron_KS33_Hotswap:Gateron-KS33-Hotswap-1U"
+		(property "Footprint" "MX_KS33:MX_KS33-Solderable-1U"
 			(at 38.1 88.9 0)
 			(effects
@@
 			)
 		)
-		(property "Footprint" "Gateron_KS33_Hotswap:Gateron-KS33-Hotswap-1U"
+		(property "Footprint" "MX_KS33:MX_KS33-Solderable-1U"
 			(at 76.2 165.1 0)
 			(effects
@@
 			)
 		)
-		(property "Footprint" "Gateron_KS33_Hotswap:Gateron-KS33-Hotswap-1U"
+		(property "Footprint" "MX_KS33:MX_KS33-Solderable-1U"
 			(at 38.1 63.5 0)
 			(effects
@@
 			)
 		)
-		(property "Footprint" "Gateron_KS33_Hotswap:Gateron-KS33-Hotswap-1U"
+		(property "Footprint" "MX_KS33:MX_KS33-Solderable-1U"
 			(at 101.6 63.5 0)
 			(effects
@@
 			)
 		)
-		(property "Footprint" "Gateron_KS33_Hotswap:Gateron-KS33-Hotswap-1U"
+		(property "Footprint" "MX_KS33:MX_KS33-Solderable-1U"
 			(at 76.2 38.1 0)
 			(effects
@@
 			)
 		)
-		(property "Footprint" "Gateron_KS33_Hotswap:Gateron-KS33-Hotswap-1U"
+		(property "Footprint" "MX_KS33:MX_KS33-Solderable-1U"
 			(at 25.4 63.5 0)
 			(effects
@@
 			)
 		)
-		(property "Footprint" "Gateron_KS33_Hotswap:Gateron-KS33-Hotswap-1U"
+		(property "Footprint" "MX_KS33:MX_KS33-Solderable-1U"
 			(at 50.8 88.9 0)
 			(effects
@@
 			)
 		)
-		(property "Footprint" "Gateron_KS33_Hotswap:Gateron-KS33-Hotswap-1U"
+		(property "Footprint" "MX_KS33:MX_KS33-Solderable-1U"
 			(at 50.8 114.3 0)
 			(effects
@@
 			)
 		)
-		(property "Footprint" "Gateron_KS33_Hotswap:Gateron-KS33-Hotswap-1U"
+		(property "Footprint" "MX_KS33:MX_KS33-Solderable-1U"
 			(at 63.5 114.3 0)
 			(effects
@@
 			)
 		)
-		(property "Footprint" "Gateron_KS33_Hotswap:Gateron-KS33-Hotswap-1.5U"
+		(property "Footprint" "MX_KS33:MX_KS33-Solderable-1.5U"
 			(at 101.6 165.1 0)
 			(effects
@@
 			)
 		)
-		(property "Footprint" "Gateron_KS33_Hotswap:Gateron-KS33-Hotswap-1U"
+		(property "Footprint" "MX_KS33:MX_KS33-Solderable-1U"
 			(at 50.8 139.7 0)
 			(effects

Commit message: Save
Checked right PCB and hole to track spacing for left. Will do check for left pcb tomorrow
Parts:
- S35, S36: footprint MX_KS33:MX_KS33-Solderable-1.5U -> MX_KS33:MX_KS33-Solderable-1.5U-Vertical
Changed lines of the file:
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@@
 			)
 		)
-		(property "Footprint" "MX_KS33:MX_KS33-Solderable-1.5U"
+		(property "Footprint" "MX_KS33:MX_KS33-Solderable-1.5U-Vertical"
 			(at 88.9 165.1 0)
 			(effects
@@
 			)
 		)
-		(property "Footprint" "MX_KS33:MX_KS33-Solderable-1.5U"
+		(property "Footprint" "MX_KS33:MX_KS33-Solderable-1.5U-Vertical"
 			(at 101.6 165.1 0)
 			(effects

Commit message: Files ready for production
Going to panelise seperate files to reduce PCBA cost
Parts:
- D1: footprint Diode_SMD:Nexperia_CFP3_SOD-123W -> Diode_SMD:D_SOD-123; LCSC Part Number (none) -> C2099
- D10, D11, D12, D13, D14, D15, D16, D17, D18, D19, D2, D20, D21, D22, D23, D24, D25, D26, D27, D28, D29, D3, D30, D31, D32, D33, D36, D37, D38, D4, D5, D6, D7, D8, D9: LCSC Part Number (none) -> C2099
