File: TheFalcon/PCB/TheFalcon[Right]/RGBArray.kicad_sch (KiCad schematic)
At the start: 61 parts, among them IC1 IS31FL3729-QFLS4-TR

Commit message: save
Parts:
- removed R17, R18: 2k, symbol Device:R
- added J6: Conn_01x01, Connector_Wire:SolderWire-0.1sqmm_1x01_D0.4mm_OD1mm, symbol Connector_Generic:Conn_01x01
- added R28: 0, Resistor_SMD:R_0805_2012Metric, symbol Device:R
- C15: renamed from C1; value 0.1u -> 100n; footprint (none) -> Capacitor_SMD:C_0603_1608Metric
- C16: renamed from C2; footprint (none) -> Capacitor_SMD:C_0603_1608Metric
- C17: renamed from C3; value 0.1u -> 100n; footprint (none) -> Capacitor_SMD:C_0603_1608Metric
- R12: renamed from R1; footprint (none) -> Resistor_SMD:R_0201_0603Metric
- R13: renamed from R2; footprint (none) -> Resistor_SMD:R_0201_0603Metric
- R14: renamed from R3; footprint (none) -> Resistor_SMD:R_0201_0603Metric
- R15: renamed from R4; footprint (none) -> Resistor_SMD:R_0201_0603Metric
- R16: renamed from R5; footprint (none) -> Resistor_SMD:R_0201_0603Metric
- R17: renamed from R6; footprint (none) -> Resistor_SMD:R_0201_0603Metric
- R18: renamed from R7; footprint (none) -> Resistor_SMD:R_0201_0603Metric
- R19: renamed from R8; footprint (none) -> Resistor_SMD:R_0201_0603Metric
- R20: renamed from R12; footprint (none) -> Resistor_SMD:R_0201_0603Metric
- R21: renamed from R13; footprint (none) -> Resistor_SMD:R_0201_0603Metric
- R22: renamed from R9; footprint (none) -> Resistor_SMD:R_0201_0603Metric
- R23: renamed from R10; footprint (none) -> Resistor_SMD:R_0201_0603Metric
- R24: renamed from R15; footprint (none) -> Resistor_SMD:R_0201_0603Metric
- R25: renamed from R14; footprint (none) -> Resistor_SMD:R_0201_0603Metric
- R26: renamed from R11; footprint (none) -> Resistor_SMD:R_0201_0603Metric
- R27: renamed from R16; footprint (none) -> Resistor_SMD:R_0201_0603Metric
- R29: renamed from R19; footprint (none) -> Resistor_SMD:R_0201_0603Metric
Connections:
- net +5V: now also R28.2
- net GND: now also J6.1 (Pin_1); no longer IC1.28 (AD)
- net R_RGB_ROW_0: now reaches R21.1, RGB13.1 (K_R), RGB18.1 (K_R), RGB23.1 (K_R), RGB28.1 (K_R), RGB3.1 (K_R), RGB33.1 (K_R), RGB36.1 (K_R), RGB8.1 (K_R)
- net R_RGB_ROW_0: now also R14.1, R17.1, R19.1, R23.1, RGB1.1 (K_R), RGB10.1 (K_R), RGB11.1 (K_R), RGB12.1 (K_R), RGB14.1 (K_R), RGB15.1 (K_R), RGB16.1 (K_R), RGB17.1 (K_R), RGB19.1 (K_R), RGB2.1 (K_R), RGB20.1 (K_R), RGB21.1 (K_R), RGB22.1 (K_R), RGB24.1 (K_R), RGB25.1 (K_R), RGB26.1 (K_R), RGB27.1 (K_R), RGB29.1 (K_R), RGB30.1 (K_R), RGB31.1 (K_R), RGB32.1 (K_R), RGB34.1 (K_R), RGB35.1 (K_R), RGB37.1 (K_R), RGB38.1 (K_R), RGB4.1 (K_R), RGB5.1 (K_R), RGB6.1 (K_R), RGB7.1 (K_R), RGB9.1 (K_R)
- net B_RGB_ROW_2: now reaches R26.1, RGB13.3 (K_B), RGB18.3 (K_B), RGB23.3 (K_B), RGB28.3 (K_B), RGB3.3 (K_B), RGB33.3 (K_B), RGB36.3 (K_B), RGB8.3 (K_B)
- net G_RGB_ROW_2: now reaches R20.1, RGB13.4 (K_G), RGB18.4 (K_G), RGB23.4 (K_G), RGB28.4 (K_G), RGB3.4 (K_G), RGB33.4 (K_G), RGB36.4 (K_G), RGB8.4 (K_G)
- net B_RGB_ROW_0: now reaches R12.1, RGB1.3 (K_B), RGB11.3 (K_B), RGB16.3 (K_B), RGB21.3 (K_B), RGB26.3 (K_B), RGB31.3 (K_B), RGB6.3 (K_B)
- net G_RGB_ROW_0: now reaches R13.1, RGB1.4 (K_G), RGB11.4 (K_G), RGB16.4 (K_G), RGB21.4 (K_G), RGB26.4 (K_G), RGB31.4 (K_G), RGB6.4 (K_G)
- net B_RGB_ROW_3: now reaches R24.1, RGB14.3 (K_B), RGB19.3 (K_B), RGB24.3 (K_B), RGB29.3 (K_B), RGB34.3 (K_B), RGB37.3 (K_B), RGB4.3 (K_B), RGB9.3 (K_B)
- net G_RGB_ROW_3: now reaches R22.1, RGB14.4 (K_G), RGB19.4 (K_G), RGB24.4 (K_G), RGB29.4 (K_G), RGB34.4 (K_G), RGB37.4 (K_G), RGB4.4 (K_G), RGB9.4 (K_G)
- net B_RGB_ROW_4: now reaches R25.1, RGB10.3 (K_B), RGB15.3 (K_B), RGB20.3 (K_B), RGB25.3 (K_B), RGB30.3 (K_B), RGB35.3 (K_B), RGB38.3 (K_B), RGB5.3 (K_B)
- net G_RGB_ROW_4: now reaches R18.1, RGB10.4 (K_G), RGB15.4 (K_G), RGB20.4 (K_G), RGB25.4 (K_G), RGB30.4 (K_G), RGB35.4 (K_G), RGB38.4 (K_G), RGB5.4 (K_G)
- net B_RGB_ROW_1: now reaches R15.1, RGB12.3 (K_B), RGB17.3 (K_B), RGB2.3 (K_B), RGB22.3 (K_B), RGB27.3 (K_B), RGB32.3 (K_B), RGB7.3 (K_B)
- net G_RGB_ROW_1: now reaches R16.1, RGB12.4 (K_G), RGB17.4 (K_G), RGB2.4 (K_G), RGB22.4 (K_G), RGB27.4 (K_G), RGB32.4 (K_G), RGB7.4 (K_G)
- new net AD: IC1.28 (AD), R28.1
Other:
- note added: "Header pin to solder AD to change address"
- note removed: "I2C Need to check if SDB, SCL and SDA need to be matched"
- note removed: "Must be 3.3V pull up 2k @ 1Mhz 4.7k @ 400kHz"
- title: (none) -> TheFalcon[Left[
- moved on the sheet: C15, C16, C17, IC1, R18, R19, R20, R21, R22, R23, R24, R25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
