File: TheFalcon/PCB/TheFalcon[Right]/TheFalcon[Right].kicad_sch (KiCad schematic)
At the start: 32 parts, among them J1 Conn_01x04_Pin, J2 Conn_02x05_Odd_Even, SW1 SW_Push, SW2 SW_Push, SW3 SW_SPDT, U1 STM32F103CBTx, U2 USBLC6-2P6, U3 USBLC6-2P6, U4 AMS1117-3.3, Y1 X322516MOB4SI

Commit message: save
Parts:
- removed FB1: 120R, symbol Device:FerriteBead
- removed R24: 1k5, symbol Device:R
- removed SW3: SW_SPDT, symbol Switch:SW_SPDT
- removed U1: STM32F103CBTx, Package_QFP:LQFP-48_7x7mm_P0.5mm, symbol MCU_ST_STM32F1:STM32F103CBTx
- added C9: 1u, Capacitor_SMD:C_0603_1608Metric, symbol Device:C
- added D1: LED, LED_SMD:LED_0805_2012Metric, symbol Device:LED
- added H1, H2, H3, H4, H5, H6: MountingHole_Pad, MountingHole:MountingHole_3.2mm_M3_Pad_Via, symbol Mechanical:MountingHole_Pad
- added J3, J4: Conn_01x01, Connector_Wire:SolderWire-0.1sqmm_1x01_D0.4mm_OD1mm, symbol Connector_Generic:Conn_01x01
- added J5: Conn_01x04_Pin, Connector_PinSocket_2.54mm:PinSocket_1x04_P2.54mm_Vertical, symbol Connector:Conn_01x04_Pin
- added R3, R8: 4k7, Resistor_SMD:R_0201_0603Metric, symbol Device:R
- added R4, R5, R6, R7: 0, Resistor_SMD:R_0805_2012Metric, symbol Device:R
- added R9: 1k5, Resistor_SMD:R_0201_0603Metric, symbol Device:R
- added SW3: SW_DIP_x02, Button_Switch_SMD:SW_DIP_SPSTx02_Slide_KingTek_DSHP02TS_W7.62mm_P1.27mm, symbol Switch:SW_DIP_x02
- added U1: STM32G431CBTx, Package_QFP:LQFP-48_7x7mm_P0.5mm, symbol MCU_ST_STM32G4:STM32G431CBTx
- added U5: USBLC6-2P6, Package_TO_SOT_SMD:SOT-666, symbol Power_Protection:USBLC6-2P6
- C1: footprint (none) -> Capacitor_SMD:C_0805_2012Metric
- C10, C11: footprint (none) -> Capacitor_SMD:C_1206_3216Metric
- C12: renamed from C9; value 0.1u -> 100n; footprint (none) -> Capacitor_SMD:C_0603_1608Metric
- C13: renamed from C15; footprint (none) -> Capacitor_SMD:C_0402_1005Metric
- C14: renamed from C16; footprint (none) -> Capacitor_SMD:C_0402_1005Metric
- C2, C3, C4, C5, C6, C7: footprint (none) -> Capacitor_SMD:C_0603_1608Metric
- C8: value 1u -> 100n; footprint (none) -> Capacitor_SMD:C_0603_1608Metric
- F1: footprint (none) -> Fuse:Fuse_1206_3216Metric
- J1: renamed from J2; footprint (none) -> Connector_PinSocket_2.54mm:PinSocket_2x05_P2.54mm_Vertical
- J2: renamed from J1; footprint (none) -> Connector_PinSocket_2.54mm:PinSocket_1x04_P2.54mm_Vertical
- R1, R2: footprint (none) -> Resistor_SMD:R_0603_1608Metric
- R10: renamed from R3; footprint (none) -> Resistor_SMD:R_0603_1608Metric
- R11: renamed from R4; footprint (none) -> Resistor_SMD:R_0603_1608Metric
- SW1: renamed from SW2; footprint (none) -> Button_Switch_SMD:SW_SPST_B3U-1000P
- SW2: renamed from SW1; footprint (none) -> Button_Switch_SMD:SW_SPST_B3U-1000P
- U2: renamed from U4; Link https://jlcpcb.com/api/file/downloadByFileSystemAccessId/85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 -> https://jlcpcb.com/partdetail/Advanced_MonolithicSystems-AM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
- USB1, USB2: Link (none) -> https://jlcpcb.com/partdetail/gswitch-GT_USB7010ASV/C2988369
- Y1: footprint X322516MOB4SI -> SamacSys_Parts:X322516MOB4SI
- renumbered U2 to U3, U3 to U4
Connections:
- net +3.3VA is gone; now on net +3.3V: C6.1, C7.1
- net +3.3V: now also C9.1, D1.2 (A), J3.1 (Pin_1), R3.1, R8.1, U1.1 (VBAT), U1.20 (VREF+), U1.21 (VDDA), U1.24 (VDD), U1.36 (VDD), U1.48 (VDD)
- net +5V: now also U5.5 (VBUS)
- net BOOT0: now also U1.45 (PB8)
- net BOOT_Tx+: now also U1.22 (PB10)
- net BOOT_Tx-: now also U1.25 (PB11)
- net Col0: now also U1.2 (PC13)
- net Col1: now also U1.3 (PC14)
- net Col2: now also U1.4 (PC15)
- net Col3: now also U1.9 (PA1)
- net Col4: now also U1.10 (PA2)
- net Col5: now also U1.11 (PA3)
- net Col6: now also U1.12 (PA4)
- net GND: now also C9.2, H1.1, H2.1, H3.1, H4.1, H5.1, H6.1, J4.1 (Pin_1), R9.1, U1.19 (VSSA), U1.23 (VSS), U1.35 (VSS), U1.47 (VSS), U5.2 (GND); no longer USB1.S1 (SHIELD), USB2.S1 (SHIELD)
- net LED_MCU_SCL: now also R8.2, SW3.3, U1.31 (PA9)
- net LED_MCU_SDA: now also R3.2, SW3.4, U1.30 (PA8)
- net LED_MCU_SDB: now also U1.32 (PA10)
- net NRST: now also U1.7 (PG10)
- net RCC_OSC_IN: now also U1.5 (PF0)
- net RCC_OSC_OUT: now also U1.6 (PF1)
- net Row0: now also U1.13 (PA5)
- net Row1: now also U1.14 (PA6)
- net Row2: now also U1.15 (PA7)
- net Row3: now also U1.16 (PB0)
- net Row4: now also U1.17 (PB1)
- net SYS_JTAG_SWCLK: now also U1.38 (PA14)
- net SYS_JTAG_SWDIO: now also U1.37 (PA13)
- net SYS_JTAG_TRACE: now also U1.40 (PB3)
- net ThumbRow: now also U1.18 (PB2)
- net USB_MCU_D+: now also U1.34 (PA12)
- net USB_MCU_D-: now also U1.33 (PA11)
- net USB_Tx+: now also U1.43 (PB6)
- net at USB2.A5 (CC1): now also R4.2
- net at USB2.A8 (SBU1): now also R6.2
- net at USB2.B5 (CC2): now also R5.2
- net at USB2.B8 (SBU2): now also R7.2
- net UBS_Tx- renamed USB_Tx-
- net USB_Tx-: now also U1.44 (PB7)
- new net I2C_DIP_SCL: SW3.2, U5.4 (I/O2)
- new net I2C_DIP_SDA: SW3.1, U5.6 (I/O1)
- new net PB12: J5.1 (Pin_1), U1.26 (PB12)
- new net PB13: J5.2 (Pin_2), U1.27 (PB13)
- new net PB14: J5.3 (Pin_3), U1.28 (PB14)
- new net PB15: J5.4 (Pin_4), U1.29 (PB15)
- new net PWR_LED: D1.1 (K), R9.2
- new net USB_CONN_SCL: R4.1, R5.1, U5.3 (I/O2)
- new net USB_CONN_SDA: R6.1, R7.1, U5.1 (I/O1)
- no-connect marks 24 -> 11
Other:
- note added: "0 Ohm resistors to disconnect I2C lines if needed"
- note added: "DONE - Change address for RGB driver on right DONE - Change Rx Tx swapover to be straight on right"
- note added: "Dip switch to disconnect I2C lines if needed"
- note added: "Enter boot by applying pattern 15: BOOT_LOCK(bit)=0, Boot0(pin) = 1, nBoot1(bit) = 1 and nBoot0_SW(bit) = 1 BOOT_LOCK(bit)=0, nBoot0(bit) = 0, nBoot1(bit) = 1 and nBoot0_SW(bit) = 0"
- note added: "I2C Connection between boards for RGB"
- note added: "MCU Breakout Points"
- note added: "Must be 3.3V pull up 2k @ 1Mhz 4.7k @ 400kHz"
- note added: "Need to check to make sure the power caps are ceramic"
- note added: "Power and Ground Breakouts"
- note added: "Tx+=Tx Tx-=Rx"
- note removed: "Need to calculate fuse value? See phils lab #11 Also need to ensure that the capacitors work for level converter. Maybe need to filter the output"
- note removed: "PA10=HIGH(LEFT) PA10=LOW(RIGHT) Might not need as I could just flash seperate files to either side"
- moved on the sheet: C1, C10, C11, C12, C13, C14, C2, C3, C4, C5, C6, C7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
