File: TheFalcon/PCB/TheFalcon[Right]/_autosave-TheFalcon[Right].kicad_sch (KiCad schematic)
At the start: 45 parts, among them J1 Conn_01x01, J2 Conn_01x04_Pin, J3 Conn_01x01, J4 Conn_01x01, J5 Conn_01x01, J7 Conn_01x01, SW1 SW_Push, SW2 SW_Push, U2 USBLC6-2P6, U3 USBLC6-2P6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

Commit message: Save
Parts:
- renumbered C2 to C12, C9 to C13, C3 to C14, C1 to C9, J3 to J2, J4 to J3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
