File: TheFalcon/PCB/TheFalcon_Panel/TheFalcon_Panel/RGBArray.kicad_sch (KiCad schematic)
At the start: 57 parts, among them IC1 IS31FL3729-QFLS4-TR

Commit message: Save
Trying a different panel
Parts:
- R10, R12, R14, R15, R17, R18, R20, R21, R23, R9: value 20 -> k020
- R11, R13, R16, R19, R22: value 51 -> k051
Changed lines of the file:
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@@
 			)
 		)
-		(property "Value" "51"
+		(property "Value" "k051"
 			(at 110.744 190.246 90)
 			(effects
@@
 			)
 		)
-		(property "Value" "20"
+		(property "Value" "k020"
 			(at 101.346 31.242 90)
 			(effects
@@
 			)
 		)
-		(property "Value" "20"
+		(property "Value" "k020"
 			(at 104.394 53.086 90)
 			(effects
@@
 			)
 		)
-		(property "Value" "51"
+		(property "Value" "k051"
 			(at 112.014 124.206 90)
 			(effects
@@
 			)
 		)
-		(property "Value" "20"
+		(property "Value" "k020"
 			(at 112.014 119.126 90)
 			(effects
@@
 			)
 		)
-		(property "Value" "20"
+		(property "Value" "k020"
 			(at 103.886 64.262 90)
 			(effects
@@
 			)
 		)
-		(property "Value" "51"
+		(property "Value" "k051"
 			(at 105.664 89.916 90)
 			(effects
@@
 			)
 		)
-		(property "Value" "20"
+		(property "Value" "k020"
 			(at 111.506 164.592 90)
 			(effects
@@
 			)
 		)
-		(property "Value" "20"
+		(property "Value" "k020"
 			(at 112.014 152.146 90)
 			(effects
@@
 			)
 		)
-		(property "Value" "51"
+		(property "Value" "k051"
 			(at 104.394 58.166 90)
 			(effects
@@
 			)
 		)
-		(property "Value" "20"
+		(property "Value" "k020"
 			(at 110.744 185.166 90)
 			(effects
@@
 			)
 		)
-		(property "Value" "51"
+		(property "Value" "k051"
 			(at 112.014 157.226 90)
 			(effects
@@
 			)
 		)
-		(property "Value" "20"
+		(property "Value" "k020"
 			(at 111.506 130.302 90)
 			(effects
@@
 			)
 		)
-		(property "Value" "20"
+		(property "Value" "k020"
 			(at 105.664 84.836 90)
 			(effects
@@
 			)
 		)
-		(property "Value" "20"
+		(property "Value" "k020"
 			(at 114.046 93.472 90)
 			(effects
