File: TheFalcon/PCB/TheFalcon_Panel/TheFalcon_Panel/RGBArray_Right.kicad_sch (KiCad schematic)
At the start: 59 parts

Commit message: Save
Trying a different panel
Parts:
- R_R1, R_R11, R_R12, R_R14, R_R15, R_R17, R_R18, R_R20, R_R21, R_R9: value 20 -> k020
- R_R10, R_R13, R_R16, R_R19, R_R22: value 51 -> k051
- R_R23: value 0 -> k0
Changed lines of the file:
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@@
 			)
 		)
-		(property "Value" "51"
+		(property "Value" "k051"
 			(at 110.744 187.706 90)
 			(effects
@@
 			)
 		)
-		(property "Value" "20"
+		(property "Value" "k020"
 			(at 101.346 28.702 90)
 			(effects
@@
 			)
 		)
-		(property "Value" "20"
+		(property "Value" "k020"
 			(at 104.394 50.546 90)
 			(effects
@@
 			)
 		)
-		(property "Value" "0"
+		(property "Value" "k0"
 			(at 210.82 39.37 90)
 			(effects
@@
 			)
 		)
-		(property "Value" "51"
+		(property "Value" "k051"
 			(at 112.014 121.666 90)
 			(effects
@@
 			)
 		)
-		(property "Value" "20"
+		(property "Value" "k020"
 			(at 112.014 116.586 90)
 			(effects
@@
 			)
 		)
-		(property "Value" "20"
+		(property "Value" "k020"
 			(at 103.886 61.722 90)
 			(effects
@@
 			)
 		)
-		(property "Value" "51"
+		(property "Value" "k051"
 			(at 105.664 87.376 90)
 			(effects
@@
 			)
 		)
-		(property "Value" "20"
+		(property "Value" "k020"
 			(at 111.506 162.052 90)
 			(effects
@@
 			)
 		)
-		(property "Value" "20"
+		(property "Value" "k020"
 			(at 112.014 149.606 90)
 			(effects
@@
 			)
 		)
-		(property "Value" "51"
+		(property "Value" "k051"
 			(at 104.394 55.626 90)
 			(effects
@@
 			)
 		)
-		(property "Value" "20"
+		(property "Value" "k020"
 			(at 110.744 182.626 90)
 			(effects
@@
 			)
 		)
-		(property "Value" "51"
+		(property "Value" "k051"
 			(at 112.014 154.686 90)
 			(effects
@@
 			)
 		)
-		(property "Value" "20"
+		(property "Value" "k020"
 			(at 111.506 127.762 90)
 			(effects
@@
 			)
 		)
-		(property "Value" "20"
+		(property "Value" "k020"
 			(at 105.664 82.296 90)
 			(effects
@@
 			)
 		)
-		(property "Value" "20"
+		(property "Value" "k020"
 			(at 114.046 90.932 90)
 			(effects
