File: TheFalcon/PCB/TheFalcon_Panel/TheFalcon_Panel/TheFalcon_Left.kicad_sch (KiCad schematic)
At the start: 39 parts, among them J1 Conn_01x01, J2 Conn_01x04_Pin, J3 Conn_01x01, J4 Conn_01x01, J5 Conn_01x01, J6 Conn_01x01, J7 Conn_01x01, SW1 SW_Push, SW2 SW_Push, U2 USBLC6-2P6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

Commit message: Save
Trying a different panel
Parts:
- added mouse-bite-1, mouse-bite-2, mouse-bite-3, mouse-bite-4, mouse-bite-5, mouse-bite-6, mouse-bite-7, mouse-bite-8: mb, Panelization.pretty-master:mouse-bite-5mm-slo-nosilk, symbol Mechanical:MountingHole

Commit message: Save
Parts:
- added mouse-bite-10, mouse-bite-11, mouse-bite-12, mouse-bite-13, mouse-bite-9: mb, Panelization.pretty-master:mouse-bite-5mm-slo-nosilk, symbol Mechanical:MountingHole
Other:
- moved on the sheet: mouse-bite-1, mouse-bite-2, mouse-bite-3, mouse-bite-4, mouse-bite-5, mouse-bite-6, mouse-bite-7
