File: TheFalcon/PCB/TheFalcon_Panel/TheFalcon_Panel/TheFalcon_Right.kicad_sch (KiCad schematic)
At the start: 35 parts

Commit message: Save
Trying a different panel
Parts:
- added R_mouse-bite-1, R_mouse-bite-2, R_mouse-bite-3, R_mouse-bite-4, R_mouse-bite-5, R_mouse-bite-6, R_mouse-bite-7, R_mouse-bite-8: mb, Panelization.pretty-master:mouse-bite-5mm-slo-nosilk, symbol Mechanical:MountingHole

Commit message: Save
Parts:
- added R_mouse-bite-10, R_mouse-bite-11, R_mouse-bite-12, R_mouse-bite-13, R_mouse-bite-9: mb, Panelization.pretty-master:mouse-bite-5mm-slo-nosilk, symbol Mechanical:MountingHole
Other:
- moved on the sheet: R_mouse-bite-1, R_mouse-bite-2, R_mouse-bite-3, R_mouse-bite-4, R_mouse-bite-5, R_mouse-bite-6, R_mouse-bite-7
