File: TheFalcon/PCB/TheFalcon_Panel/TheFalcon_Panel/TheFalcon_Panel.kicad_pcb (KiCad board)
At the start: 4 copper layers, 185.7 x 303.9 mm, 362 parts, among them IC1 IS31FL3729-QFLS4-TR, J1 Conn_01x01, J2 Conn_01x04_Pin, J3 Conn_01x01, J4 Conn_01x01, J5 Conn_01x01, J6 Conn_01x01, J7 Conn_01x01, SW1 SW_Push, SW2 SW_Push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

Commit message: Save
Routing:
- net /Right/RGB Array/R_SW7: track 138.1 -> 140.4 mm
- net /Right/RGB Array/R_SW2: track 124.9 -> 125.9 mm
- net /Left/RGB Array/SW3: track 138.5 -> 137.7 mm
- net /Right/RGB Array/R_SW8: track 123.1 -> 123.6 mm
